File: kicad/as3340/output_mix.sch (KiCad schematic (older format))
At the start: 21 parts, among them U1 TL074, U5 DG442CY+, U6 AS3360, U8 DG442CY+

Commit message: testing...
Parts:
- removed R66: 1k, Resistor_SMD:R_0603_1608Metric, symbol Device:R
- R10: value 100k -> 1k; LCSC Part \\ -> (none)
- R2, R3, R5: value 47k -> 51k; LCSC Part C25819 -> (none)
- R39: value 50k -> 51k
- R59: value 33k -> 51k
- R6: value 100k -> 200k
- R7: value 50k -> 100k
- R70: value 100k -> 51k
- R8: LCSC Part C23196 -> (none)
- R9: value 200k -> 100k
Connections:
- net GND: no longer R59.2
- net MIX1_INV: now also R59.1, U5.15, U5.2, U5.6; no longer R10.2, R39.1, U5.11
- net MIX1_NONINV: now also R39.1, U5.11; no longer R59.1, U5.15, U5.2, U5.6
- net OSC1_MIX1: now also R10.2
- net TRI_VC_AMOUNT_DAC: now also R59.2; no longer R2.2
- net at R70.2, U1.8: now also R2.2
- net MIX1_SAW_CTRL renamed MIX1_SAW_LEVEL_CTRL2
- net SAW_LEVEL_CTRL renamed MIX1_SAW_LEVEL_CTRL1
Other:
- moved on the sheet: R10, R12, R2, R3, R39, R5, R6, R7, R70, R8, R9, U1C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

Commit message: routed for v0.3 -- perhaps final
Parts:
- removed U5: DG442CY+, Package_SO:SOIC-16_3.9x9.9mm_P1.27mm, symbol Analog_Switch:DG441xJ
- added C38, C40: 22p, Capacitor_SMD:C_0603_1608Metric, symbol Device:C
- added R66, R71, R73: 47k, Resistor_SMD:R_0603_1608Metric, symbol Device:R
- added R72: 180k, Resistor_SMD:R_0603_1608Metric, symbol Device:R
- added R74: 560k, Resistor_SMD:R_0603_1608Metric, symbol Device:R
- added R75: 360k, Resistor_SMD:R_0603_1608Metric, symbol Device:R
- added unit 2 of U1
- added U5: MAX333A, symbol Analog_Switch:MAX333A
- R11: value 560k -> 100k
- R12: value 100k -> 120k
- R13: value 27k -> 150k; LCSC Part C22967 -> (none)
- R14: value 20k -> 100k; LCSC Part C4184 -> (none)
- R2, R3, R39, R5, R70, R8: value 51k -> 47k
- R59: value 51k -> 24k
- R6: value 200k -> 62k
- R7: value 100k -> 120k; LCSC Part (none) -> C25808
- R9: value 100k -> 150k
Connections:
- net GND: now also U1.3 (+), U1.5 (+), U5.14, U5.17, U5.4, U5.7
- net MIX1_COMP_OSC2_CTRL: now also U5.11
- net MIX1_INV: now also C38.2, U5.12, U5.19, U5.2, U5.9
- net MIX1_PULSE_CTRL: now also U5.20
- net MIX1_SAW_LEVEL_CTRL1: now also U5.1
- net MIX1_SAW_LEVEL_CTRL2: now also U5.10
- net at R9.2: now also R74.2, U5.18
- net at R12.2: now also U5.13
- net at R11.1, R13.2, R14.2: now also U1.2 (-), C40.2, R66.1; no longer U1.3 (+)
- net at R2.2, R70.2, U1.8: now also C38.1
- net at R6.2: now also R72.2, U5.8
- net at R7.2: now also R75.2, U5.3
- new net: R65.1, R73.1, U1.7
- new net: C40.1, R66.2, R71.2, U1.1
- new net: R71.1, R73.2, U1.6 (-)
- new net -12V: R72.1, R74.1, R75.1
Other:
- note added: "I don’t think R39 is required…"
- note added: "Mix1\nSignal Input Level Output: Offset Low High Peak-to-Peak\nPulse -3 : 10.5 -1 -2 2.3 4.3\nSaw1 0 : 8 -1.5 -1.5 1.5 3\nSaw2 0 : 8 -3 -3 3 6\nTriangle 0 : 4 -4 -4 4 8\nComparator -5 : 5 0 -2 2 4\n\nand how do I get a fixed width font?"
- note removed: "TODO: REVIEW PRO-ONE AS AN EXAMPLE MIX\nTODO: REVERT OUTPUT AMPLIFICATION TO V0.2 LEVEL"
- moved on the sheet: R10, R11, R12, R13, R14, R2, R3, R39, R5, R6, R65, R7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

Commit message: update gerber files and assembly
Parts:
- removed R39: 47k, Resistor_SMD:R_0603_1608Metric, symbol Device:R
- C38, C40: LCSC Part (none) -> C1653
- R10, R65: LCSC Part (none) -> C21190
- R11, R14: LCSC Part (none) -> C25803
- R12: LCSC Part \\ -> C25808
- R13: LCSC Part (none) -> C22807
- R2, R3, R5, R66, R70, R71, R73, R8: LCSC Part (none) -> C25819
- R59: LCSC Part (none) -> C23352
- R6: LCSC Part (none) -> C23221
- R72: LCSC Part (none) -> C22827
- R74: value 560k -> 220k; LCSC Part (none) -> C22961
- R75: LCSC Part (none) -> C23146
- R9: value 150k -> 91k; LCSC Part (none) -> C23265
Connections:
- net VCA_TRI is gone; now on net MIX1_NONINV: R8.2, U6.2 (Io)
Other:
- note added: "Mix1\nSignal Input Level Output: Offset Low High Peak-to-Peak\nPulse 0 : 10.5 -2.5 -2.5 2.5 5\nSaw1 0 : 8 -1.5 -1.5 1.5 3\nSaw2 0 : 8 -3 -3 3 6\nTriangle 0 : 4 -4 -4 4 8\nComparator -5 : 5 0 -2 2 4\n\nand how do I get a fixed width font?"
- note removed: "I don’t think R39 is required…"
- note removed: "Mix1\nSignal Input Level Output: Offset Low High Peak-to-Peak\nPulse -3 : 10.5 -1 -2 2.3 4.3\nSaw1 0 : 8 -1.5 -1.5 1.5 3\nSaw2 0 : 8 -3 -3 3 6\nTriangle 0 : 4 -4 -4 4 8\nComparator -5 : 5 0 -2 2 4\n\nand how do I get a fixed width font?"
Changed lines of the file:
@@
 AR Path="/6269DD41/626F5A6B" Ref="R9"  Part="1"
 F 0 "R9" V 9150 1150 50  0000 C CNN
-F 1 "150k" V 8950 1150 50  0000 C CNN
+F 1 "91k" V 8950 1150 50  0000 C CNN
 F 2 "Resistor_SMD:R_0603_1608Metric" V 8980 1150 50  0001 C CNN
 F 3 "~" H 9050 1150 50  0001 C CNN
-F 4 "" H 9050 1150 50  0001 C CNN "LCSC Part"
+F 4 "C23265" H 9050 1150 50  0001 C CNN "LCSC Part"
 	1    9050 1150
 	0    -1   -1   0
@@
 F 2 "Resistor_SMD:R_0603_1608Metric" V 9130 7550 50  0001 C CNN
 F 3 "~" H 9200 7550 50  0001 C CNN
-F 4 "" H 9200 7550 50  0001 C CNN "LCSC Part"
+F 4 "C22807" H 9200 7550 50  0001 C CNN "LCSC Part"
 	1    9200 7550
 	0    -1   -1   0
@@
 F 2 "Resistor_SMD:R_0603_1608Metric" V 8530 3050 50  0001 C CNN
 F 3 "~" H 8600 3050 50  0001 C CNN
-F 4 "" H 8600 3050 50  0001 C CNN "LCSC Part"
+F 4 "C23221" H 8600 3050 50  0001 C CNN "LCSC Part"
 	1    8600 3050
 	0    -1   -1   0
@@
 F 2 "Resistor_SMD:R_0603_1608Metric" V 12830 7750 50  0001 C CNN
 F 3 "~" H 12900 7750 50  0001 C CNN
-F 4 "" H 12900 7750 50  0001 C CNN "LCSC Part"
+F 4 "C21190" H 12900 7750 50  0001 C CNN "LCSC Part"
 	1    12900 7750
 	0    -1   -1   0
@@
 F 2 "Resistor_SMD:R_0603_1608Metric" V 9130 8300 50  0001 C CNN
 F 3 "~" H 9200 8300 50  0001 C CNN
-F 4 "" H 9200 8300 50  0001 C CNN "LCSC Part"
+F 4 "C25803" H 9200 8300 50  0001 C CNN "LCSC Part"
 	1    9200 8300
 	0    -1   -1   0
@@
 F 2 "Resistor_SMD:R_0603_1608Metric" V 9380 8600 50  0001 C CNN
 F 3 "~" H 9450 8600 50  0001 C CNN
-F 4 "" H 9450 8600 50  0001 C CNN "LCSC Part"
+F 4 "C25803" H 9450 8600 50  0001 C CNN "LCSC Part"
 	1    9450 8600
 	1    0    0    -1
@@
 F 2 "Resistor_SMD:R_0603_1608Metric" V 8580 5500 50  0001 C CNN
 F 3 "~" H 8650 5500 50  0001 C CNN
-F 4 "" H 8650 5500 50  0001 C CNN "LCSC Part"
+F 4 "C25819" H 8650 5500 50  0001 C CNN "LCSC Part"
 	1    8650 5500
 	0    -1   -1   0
@@
 F 2 "Resistor_SMD:R_0603_1608Metric" V 9480 5400 50  0001 C CNN
 F 3 "~" H 9550 5400 50  0001 C CNN
-F 4 "" H 9550 5400 50  0001 C CNN "LCSC Part"
+F 4 "C25819" H 9550 5400 50  0001 C CNN "LCSC Part"
 	1    9550 5400
 	-1   0    0    1
@@
 F 2 "Resistor_SMD:R_0603_1608Metric" V 11480 4200 50  0001 C CNN
 F 3 "~" H 11550 4200 50  0001 C CNN
-F 4 "" H 11550 4200 50  0001 C CNN "LCSC Part"
+F 4 "C25819" H 11550 4200 50  0001 C CNN "LCSC Part"
 	1    11550 4200
 	0    -1   -1   0
@@
 Wire Wire Line
 	12050 4200 12050 4700
-$Comp
-L Device:R R?
-U 1 1 62A68F31
-P 9900 5150
-AR Path="/61E1D4AE/62A68F31" Ref="R?"  Part="1"
-AR Path="/62A68F31" Ref="R?"  Part="1"
-AR Path="/6269DD41/62A68F31" Ref="R39"  Part="1"
-F 0 "R39" V 10000 5150 50  0000 C CNN
-F 1 "47k" V 9800 5150 50  0000 C CNN
-F 2 "Resistor_SMD:R_0603_1608Metric" V 9830 5150 50  0001 C CNN
-F 3 "~" H 9900 5150 50  0001 C CNN
-F 4 "" H 9900 5150 50  0001 C CNN "LCSC Part"
-	1    9900 5150
-	0    1    1    0
-$EndComp
 Wire Wire Line
 	10500 4600 11100 4600
@@
 F 2 "Resistor_SMD:R_0603_1608Metric" V 13130 4350 50  0001 C CNN
 F 3 "~" H 13200 4350 50  0001 C CNN
-F 4 "" H 13200 4350 50  0001 C CNN "LCSC Part"
+F 4 "C25819" H 13200 4350 50  0001 C CNN "LCSC Part"
 	1    13200 4350
 	0    1    1    0
 $EndComp
-Wire Wire Line
-	9550 5150 9750 5150
 Connection ~ 9550 5150
 $Comp
@@
 F 2 "Resistor_SMD:R_0603_1608Metric" V 12330 4700 50  0001 C CNN
 F 3 "~" H 12400 4700 50  0001 C CNN
-F 4 "" H 12400 4700 50  0001 C CNN "LCSC Part"
+F 4 "C25819" H 12400 4700 50  0001 C CNN "LCSC Part"
 	1    12400 4700
 	0    1    1    0
@@
 F 2 "Resistor_SMD:R_0603_1608Metric" V 13830 4800 50  0001 C CNN
 F 3 "~" H 13900 4800 50  0001 C CNN
-F 4 "" H 13900 4800 50  0001 C CNN "LCSC Part"
+F 4 "C21190" H 13900 4800 50  0001 C CNN "LCSC Part"
 	1    13900 4800
 	0    -1   -1   0
@@
 F 2 "Resistor_SMD:R_0603_1608Metric" V 9130 3850 50  0001 C CNN
 F 3 "~" H 9200 3850 50  0001 C CNN
-F 4 "\\" H 9200 3850 50  0001 C CNN "LCSC Part"
+F 4 "C25808" H 9200 3850 50  0001 C CNN "LCSC Part"
 	1    9200 3850
 	0    -1   -1   0
@@
 F 2 "Capacitor_SMD:C_0603_1608Metric" H 11588 3700 50  0001 C CNN
 F 3 "~" H 11550 3850 50  0001 C CNN
-F 4 "" V 11550 3850 50  0001 C CNN "LCSC Part"
+F 4 "C1653" V 11550 3850 50  0001 C CNN "LCSC Part"
 	1    11550 3850
 	0    1    1    0
@@
 F 2 "Resistor_SMD:R_0603_1608Metric" V 10430 7150 50  0001 C CNN
 F 3 "~" H 10500 7150 50  0001 C CNN
-F 4 "" H 10500 7150 50  0001 C CNN "LCSC Part"
+F 4 "C25819" H 10500 7150 50  0001 C CNN "LCSC Part"
 	1    10500 7150
 	0    -1   -1   0
@@
 F 2 "Resistor_SMD:R_0603_1608Metric" V 12130 7300 50  0001 C CNN
 F 3 "~" H 12200 7300 50  0001 C CNN
-F 4 "" H 12200 7300 50  0001 C CNN "LCSC Part"
+F 4 "C25819" H 12200 7300 50  0001 C CNN "LCSC Part"
 	1    12200 7300
 	0    1    1    0
@@
 F 2 "Resistor_SMD:R_0603_1608Metric" V 11280 7650 50  0001 C CNN
 F 3 "~" H 11350 7650 50  0001 C CNN
-F 4 "" H 11350 7650 50  0001 C CNN "LCSC Part"
+F 4 "C25819" H 11350 7650 50  0001 C CNN "LCSC Part"
 	1    11350 7650
 	0    1    1    0
@@
 F 2 "Capacitor_SMD:C_0603_1608Metric" H 10538 6650 50  0001 C CNN
 F 3 "~" H 10500 6800 50  0001 C CNN
-F 4 "" V 10500 6800 50  0001 C CNN "LCSC Part"
+F 4 "C1653" V 10500 6800 50  0001 C CNN "LCSC Part"
 	1    10500 6800
 	0    1    1    0
@@
 F 2 "Resistor_SMD:R_0603_1608Metric" V 9830 4600 50  0001 C CNN
 F 3 "~" H 9900 4600 50  0001 C CNN
-F 4 "" H 9900 4600 50  0001 C CNN "LCSC Part"
+F 4 "C23352" H 9900 4600 50  0001 C CNN "LCSC Part"
 	1    9900 4600
 	0    1    1    0
@@
 AR Path="/6269DD41/6319A98E" Ref="R74"  Part="1"
 F 0 "R74" V 9150 700 50  0000 C CNN
-F 1 "560k" V 8950 700 50  0000 C CNN
+F 1 "220k" V 8950 700 50  0000 C CNN
 F 2 "Resistor_SMD:R_0603_1608Metric" V 8980 700 50  0001 C CNN
 F 3 "~" H 9050 700 50  0001 C CNN
-F 4 "" H 9050 700 50  0001 C CNN "LCSC Part"
+F 4 "C22961" H 9050 700 50  0001 C CNN "LCSC Part"
 	1    9050 700
 	0    -1   -1   0
@@
 F 2 "Resistor_SMD:R_0603_1608Metric" V 8980 1800 50  0001 C CNN
 F 3 "~" H 9050 1800 50  0001 C CNN
-F 4 "" H 9050 1800 50  0001 C CNN "LCSC Part"
+F 4 "C23146" H 9050 1800 50  0001 C CNN "LCSC Part"
 	1    9050 1800
 	0    -1   -1   0
@@
 F 2 "Resistor_SMD:R_0603_1608Metric" V 9130 2750 50  0001 C CNN
 F 3 "~" H 9200 2750 50  0001 C CNN
-F 4 "" H 9200 2750 50  0001 C CNN "LCSC Part"
+F 4 "C22827" H 9200 2750 50  0001 C CNN "LCSC Part"
 	1    9200 2750
 	0    -1   -1   0
@@
 	10150 3750 10300 3750
 Wire Wire Line
-	10050 5150 10400 5150
-Wire Wire Line
 	10150 3950 10500 3950
 Wire Wire Line
@@
 $EndComp
 Text Notes 12000 2000 0    50   ~ 0
-Mix1\nSignal          Input Level    Output:  Offset     Low   High       Peak-to-Peak\nPulse           -3 : 10.5                      -1          -2      2.3        4.3\nSaw1             0 : 8                         -1.5        -1.5    1.5         3\nSaw2             0 : 8                         -3         -3       3         6\nTriangle         0 : 4                         -4          -4       4            8\nComparator      -5 : 5                     0           -2       2            4\n\nand how do I get a fixed width font?
+Mix1\nSignal          Input Level    Output:  Offset     Low   High       Peak-to-Peak\nPulse           0 : 10.5                   -2.5         -2.5      2.5        5\nSaw1             0 : 8                      -1.5        -1.5    1.5         3\nSaw2             0 : 8                      -3         -3       3         6\nTriangle         0 : 4                      -4          -4       4            8\nComparator      -5 : 5                  0           -2       2            4\n\nand how do I get a fixed width font?
 Wire Notes Line
 	11900 1200 15600 1200
@@
 Wire Wire Line
 	10400 4800 11300 4800
-Text Notes 9850 5350 0    50   Italic 0
-I don’t think R39 is required…
+Wire Wire Line
+	9550 5150 10400 5150
 $EndSCHEMATC
