File: kicad/as3340/as3340.sch (KiCad schematic (older format))
At the start: 43 parts, among them J1 Conn_02x20_Odd_Even, U1 TL074, U11 LM393, U12 TL074, U2 TL074, U4 DG303B, U5 DG442CY+, U6 AS3360, U7 PCA9555D, U8 DG442CY+, U9 DG442CY+

Commit message: start revision 0.3 of board
Parts:
- removed J1: Conn_02x20_Odd_Even, Connector_PinHeader_2.54mm:PinHeader_2x20_P2.54mm_Vertical, symbol Connector_Generic:Conn_02x20_Odd_Even
- removed R11: 1k, Resistor_SMD:R_1206_3216Metric, symbol Device:R
- removed R2: 47k, Resistor_SMD:R_0603_1608Metric, symbol Device:R
- removed R3: 100k, Resistor_SMD:R_0603_1608Metric, symbol Device:R
- removed unit 4 of U12
- removed unit 4 of U8
- removed unit 1 of U9
- added C34: 0.1u, Capacitor_SMD:C_0603_1608Metric, symbol Device:C
- added J3: Conn_02x20_Odd_Even, Connector_PinHeader_2.54mm:PinHeader_2x20_P2.54mm_Vertical, symbol Connector_Generic:Conn_02x20_Odd_Even
- added R26: 510, Resistor_SMD:R_0603_1608Metric, symbol Device:R
- added unit 4 of U8
- H1, H2, H3, H4: footprint MountingHole:MountingHole_3.2mm_M3_Pad -> MountingHole:MountingHole_3.2mm_M3
- R4: value 1k -> 5k1; footprint Resistor_SMD:R_1206_3216Metric -> Resistor_SMD:R_0603_1608Metric; LCSC Part C4410 -> (none)
- U4: symbol as3340-rescue:DG303B-Analog_Switch -> Analog_Switch:DG303B
- U6: symbol as3340-rescue:AS3360-Audio -> Audio:AS3360
Connections:
- net labels added: -5V, CARD1_OUT1, CARD1_OUT2, CARD2_OUT1, CARD2_OUT2, CARD3_OUT1, CARD3_OUT2, CARD4_OUT1, CARD4_OUT2, CARD5_OUT1, CARD5_OUT2, CARD6_OUT1, CARD6_OUT2, ID_CS, SPI_CLK, SPI_CS, SPI_MISO, SPI_MOSI, SYNC_NEG_CTRL, SYNC_POS_CTRL, THIS_OUT1, THIS_OUT2
- net labels removed: EXT_CV, EXT_FREQ_CV_CTRL, FILT1_OUT1, FILT1_OUT2, FILT2_OUT1, FILT2_OUT2, FX1, FX2, GPIO_PI_DRIVEN, HARD_SYNC_CTRL, OSC1_CV, OSC1_MIX1, OSC1_MIX2, OSC2_CV, OSC2_MIX1, OSC2_MIX2, SPI0_MOSI, SPI0_SCLK, VCA1_OUT, VCA2_OUT, VCA3_OUT
- wire segments 252 -> 241
- no-connect marks 22 -> 24
Other:
- note removed: "Hardwired as Osc1: the connections below should be\nrewired to use this as Osc2.\nMaking a switchable Osc1/Osc2 isn’t in scope"
- note removed: "Osc CVs"
- note removed: "TODO: REVIEW OVERVOLTAGE"
- moved on the sheet: C32, D3, R4, U1B, U8B

Commit message: routed v0.3
Parts:
- removed U4: DG303B, Package_SO:SOIC-14_3.9x8.7mm_P1.27mm, symbol Analog_Switch:DG303B
- removed unit 2 of U8
- added C36, C37: 0.1u, Capacitor_SMD:C_0603_1608Metric, symbol Device:C
- added R60: 100k, Resistor_SMD:R_0603_1608Metric, symbol Device:R
- added U15: 74HC165, Package_SO:SOIC-16_3.9x9.9mm_P1.27mm, symbol 74xx:74HC165
- added unit 2 of U2
- added U4: PS508, Package_SO:SOIC-16_3.9x9.9mm_P1.27mm, symbol Analog_Switch:PS508
Connections:
- net labels added: EXT_MOD_SEL_CTRL0, EXT_MOD_SEL_CTRL1, EXT_MOD_SEL_CTRL2
- net labels removed: EXT_MOD_SEL_CTRL
- wire segments 241 -> 277
- no-connect marks 24 -> 15
Other:
- note added: "Board ID - can be read in SPI mode 0"
- moved on the sheet: C1, C10, C11, C12, C2, C26, C27, C28, C29, C3, C30, C31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

Commit message: testing...
Connections:
- net labels added: MIX1_SAW_LEVEL_CTRL1, MIX1_SAW_LEVEL_CTRL2
- net labels removed: MIX1_SAW_CTRL, SAW_LEVEL_CTRL
- wire segments 277 -> 284
- no-connect marks 15 -> 12
Other:
- note added: "Program control signals"
- note removed: "Logic control signals"
- moved on the sheet: C13, D4, R56, U7

Commit message: routed for v0.3 -- perhaps final
Parts:
- removed unit 2 of U1
- removed U5: DG442CY+, Package_SO:SOIC-16_3.9x9.9mm_P1.27mm, symbol Analog_Switch:DG441xJ
- added D5: 1N5819WS, Diode_SMD:D_SOD-323, symbol Diode:1N4148W
- added U5: MAX333A, Package_SO:SOIC-20W_7.5x12.8mm_P1.27mm, symbol Analog_Switch:MAX333A
- D3: value 1N4148W -> 1N5819WS; footprint Diode_SMD:D_SOD-123 -> Diode_SMD:D_SOD-323; LCSC Part C81598 -> C191023
Connections:
- wire segments 284 -> 279
Other:
- note added: "DG442: Ensure model is spec’d for +/- 12V. LE is not\nMAX333A: MAX333AEWP+ or MAX333ACWP+"
- note removed: "DG442: Ensure model is spec’d for +/- 12V. LE is not."
- moved on the sheet: U2B
Changed lines of the file:
@@
 L power:GND #PWR019
 U 1 1 61EA96D1
-P 5500 10050
-F 0 "#PWR019" H 5500 9800 50  0001 C CNN
-F 1 "GND" H 5505 9877 50  0000 C CNN
-F 2 "" H 5500 10050 50  0001 C CNN
-F 3 "" H 5500 10050 50  0001 C CNN
-	1    5500 10050
+P 5600 10050
+F 0 "#PWR019" H 5600 9800 50  0001 C CNN
+F 1 "GND" H 5605 9877 50  0000 C CNN
+F 2 "" H 5600 10050 50  0001 C CNN
+F 3 "" H 5600 10050 50  0001 C CNN
+	1    5600 10050
 	1    0    0    -1
 $EndComp
@@
 Wire Wire Line
 	7800 2050 7850 2050
+Text Label 7850 2350 0    50   ~ 0
+EXP_FM_EXT_CTRL
 Text Label 7850 2550 0    50   ~ 0
-EXP_FM_EXT_CTRL
-Text Label 7850 2350 0    50   ~ 0
 LINEAR_FM_EXT_CTRL
 Text Label 7850 2450 0    50   ~ 0
@@
 Text Label 14500 8250 2    50   ~ 0
 GPIO_MODULE_DRIVEN
-Text Notes 10900 7650 0    50   ~ 10
+Text Notes 10900 7550 0    50   ~ 10
 Tune Control: send pulse back to Pi for freq count
 $Comp
@@
 	7800 3250 7850 3250
 Wire Notes Line
-	600  10400 600  8450
-Wire Notes Line
 	14950 7100 16500 7100
 Wire Notes Line
 	16500 7100 16500 9200
-Wire Wire Line
-	12000 8150 12000 7900
-Wire Wire Line
-	12000 8150 12100 8150
 $Comp
 L Device:R R?
@@
 $EndComp
 Wire Notes Line
-	600  10400 9400 10400
+	600  10450 9400 10450
 Wire Notes Line
 	600  8450 9400 8450
-Wire Notes Line
-	9400 8450 9400 10400
 $Comp
 L power:GND #PWR0114
@@
 	6700 9900 6700 9800
 $Comp
-L Analog_Switch:DG441xJ U5
-U 5 1 6220D436
-P 5500 9300
-F 0 "U5" H 5500 9350 50  0000 L CNN
-F 1 "DG442CY+" H 5400 9250 50  0000 L CNN
-F 2 "Package_SO:SOIC-16_3.9x9.9mm_P1.27mm" H 5500 9200 50  0001 C CNN
-F 3 "https://datasheets.maximintegrated.com/en/ds/DG441-DG442.pdf" H 5500 9300 50  0001 C CNN
-F 4 "DG442CY+-ND" H 5500 9300 50  0001 C CNN "Digikey"
-	5    5500 9300
-	1    0    0    -1
-$EndComp
-$Comp
 L power:GND #PWR017
 U 1 1 6393A1F0
@@
 Connection ~ 5050 9200
 Wire Wire Line
-	5500 9800 5500 10050
+	5600 9800 5600 10050
 $Comp
 L power:GND #PWR025
@@
 Wire Wire Line
 	5050 9200 5200 9200
-Connection ~ 5600 9900
-Wire Wire Line
-	5050 9900 5600 9900
+Connection ~ 5500 9900
 Wire Wire Line
 	5050 9650 5050 9900
@@
 L power:-12V #PWR?
 U 1 1 61F6A66B
-P 5600 9900
+P 5500 9900
 AR Path="/61FF2290/61F6A66B" Ref="#PWR?"  Part="1"
 AR Path="/61F6A66B" Ref="#PWR020"  Part="1"
-F 0 "#PWR020" H 5600 10000 50  0001 C CNN
-F 1 "-12V" H 5615 10073 50  0000 C CNN
-F 2 "" H 5600 9900 50  0001 C CNN
-F 3 "" H 5600 9900 50  0001 C CNN
-	1    5600 9900
+F 0 "#PWR020" H 5500 10000 50  0001 C CNN
+F 1 "-12V" H 5515 10073 50  0000 C CNN
+F 2 "" H 5500 9900 50  0001 C CNN
+F 3 "" H 5500 9900 50  0001 C CNN
+	1    5500 9900
 	-1   0    0    1
 $EndComp
@@
 $EndComp
 Wire Wire Line
-	5600 9900 5600 9800
+	5500 9900 5500 9800
 $Comp
 L Device:C C?
@@
 Wire Wire Line
 	8850 5250 8350 5250
-Text Label 11700 8350 2    50   ~ 0
+Text Label 11850 8350 2    50   ~ 0
 VCO_PULSE
 $Comp
@@
 P 13250 7900
 F 0 "D3" V 13204 7980 50  0000 L CNN
-F 1 "1N4148W" V 13295 7980 50  0000 L CNN
-F 2 "Diode_SMD:D_SOD-123" H 13250 7725 50  0001 C CNN
-F 3 "https://www.vishay.com/docs/85748/1n4148w.pdf" H 13250 7900 50  0001 C CNN
-F 4 "C81598" H 13250 7900 50  0001 C CNN "LCSC Part"
+F 1 "1N5819WS" V 13295 7980 50  0000 L CNN
+F 2 "Diode_SMD:D_SOD-323" H 13250 7725 50  0001 C CNN
+F 3 "" H 13250 7900 50  0001 C CNN
+F 4 "C191023" H 13250 7900 50  0001 C CNN "LCSC Part"
 	1    13250 7900
 	0    1    1    0
@@
 Wire Wire Line
 	14050 5550 13650 5550
-Text Notes 5100 10400 0    50   ~ 0
-DG442: Ensure model is spec’d for +/- 12V. LE is not.
+Text Notes 5100 10450 0    50   ~ 0
+DG442: Ensure model is spec’d for +/- 12V. LE is not\nMAX333A: MAX333AEWP+ or MAX333ACWP+
 Text Label 7900 2150 0    50   ~ 0
 LED_CTRL
@@
 Wire Wire Line
 	4350 9250 4350 9500
-Wire Wire Line
-	12000 7900 12750 7900
 Wire Wire Line
 	13150 8250 13250 8250
@@
 Wire Wire Line
 	13250 8050 13250 8250
-Wire Wire Line
-	12700 8250 12750 8250
-Wire Wire Line
-	12750 7900 12750 8250
-Connection ~ 12750 8250
-Wire Wire Line
-	12750 8250 12850 8250
 Wire Wire Line
 	13700 8250 14500 8250
@@
 NoConn ~ 2750 3050
 $Comp
-L Amplifier_Operational:TL074 U?
-U 2 1 6500B008
-P 12400 8250
-AR Path="/627C7865/6500B008" Ref="U?"  Part="2"
-AR Path="/627EC897/6500B008" Ref="U?"  Part="1"
-AR Path="/63514083/6500B008" Ref="U?"  Part="2"
-AR Path="/6500B008" Ref="U1"  Part="2"
-F 0 "U1" H 12400 8450 50  0000 C CNN
-F 1 "TL074" H 12350 8250 50  0000 C CNN
-F 2 "Package_SO:SOIC-14_3.9x8.7mm_P1.27mm" H 12400 8250 50  0001 C CNN
-F 3 "http://www.ti.com/lit/ds/symlink/tl071.pdf" H 12400 8250 50  0001 C CNN
-F 4 "C12594" H 12400 8250 50  0001 C CNN "LCSC Part"
-	2    12400 8250
-	1    0    0    1
-$EndComp
-Wire Wire Line
-	11700 8350 12100 8350
-$Comp
 L power:PWR_FLAG #FLG0103
 U 1 1 62B12082
@@
 	10550 2450 10550 2300
 NoConn ~ 7850 3250
-Wire Wire Line
-	16050 7550 16150 7550
-Wire Wire Line
-	16150 7550 16150 7800
-Wire Wire Line
-	15450 7450 15250 7450
-Wire Wire Line
-	15250 7450 15250 7600
-$Comp
-L power:GND #PWR0121
-U 1 1 62B39ECF
-P 15250 7600
-F 0 "#PWR0121" H 15250 7350 50  0001 C CNN
-F 1 "GND" H 15255 7427 50  0000 C CNN
-F 2 "" H 15250 7600 50  0001 C CNN
-F 3 "" H 15250 7600 50  0001 C CNN
-	1    15250 7600
-	1    0    0    -1
-$EndComp
-Wire Wire Line
-	15400 7650 15450 7650
-Wire Wire Line
-	15400 7800 15400 7650
-Wire Wire Line
-	16150 7800 15400 7800
 $Comp
 L Amplifier_Operational:TL074 U?
 U 2 1 629F9E1F
-P 15750 7550
+P 12400 8250
 AR Path="/61E1D4AE/629F9E1F" Ref="U?"  Part="1"
 AR Path="/629F9E1F" Ref="U2"  Part="2"
-F 0 "U2" H 15850 7400 50  0000 C CNN
-F 1 "TL074" H 15700 7550 50  0000 C CNN
-F 2 "Package_SO:SOIC-14_3.9x8.7mm_P1.27mm" H 15700 7650 50  0001 C CNN
-F 3 "http://www.ti.com/lit/ds/symlink/tl071.pdf" H 15800 7750 50  0001 C CNN
-F 4 "C12594" H 15750 7550 50  0001 C CNN "LCSC Part"
-	2    15750 7550
-	1    0    0    -1
-$EndComp
+F 0 "U2" H 12500 8100 50  0000 C CNN
+F 1 "TL074" H 12350 8250 50  0000 C CNN
+F 2 "Package_SO:SOIC-14_3.9x8.7mm_P1.27mm" H 12350 8350 50  0001 C CNN
+F 3 "http://www.ti.com/lit/ds/symlink/tl071.pdf" H 12450 8450 50  0001 C CNN
+F 4 "C12594" H 12400 8250 50  0001 C CNN "LCSC Part"
+	2    12400 8250
+	1    0    0    1
+$EndComp
+Text Label 7850 2950 0    50   ~ 0
+MIX1_SAW_LEVEL_CTRL2
 Text Label 7850 3050 0    50   ~ 0
-MIX1_SAW_LEVEL_CTRL2
-Text Label 7850 2950 0    50   ~ 0
 MIX1_SAW_LEVEL_CTRL1
 $Sheet
@@
 F14 "OSC1_MIX1" O R 13650 5350 50
 $EndSheet
+$Comp
+L Analog_Switch:MAX333A U5
+U 5 1 630BCD26
+P 5500 9300
+F 0 "U5" H 5780 9346 50  0000 L CNN
+F 1 "MAX333A" H 5780 9255 50  0000 L CNN
+F 2 "Package_SO:SOIC-20W_7.5x12.8mm_P1.27mm" H 5500 9300 50  0001 C CNN
+F 3 "https://datasheets.maximintegrated.com/en/ds/MAX333A.pdf" H 5500 9300 50  0001 C CNN
+	5    5500 9300
+	1    0    0    -1
+$EndComp
+Wire Wire Line
+	5050 9900 5500 9900
+Wire Notes Line
+	9400 8450 9400 10450
+Wire Notes Line
+	600  8450 600  10450
+$Comp
+L Diode:1N4148W D5
+U 1 1 6355B1F4
+P 13250 8550
+F 0 "D5" V 13204 8630 50  0000 L CNN
+F 1 "1N5819WS" V 13295 8630 50  0000 L CNN
+F 2 "Diode_SMD:D_SOD-323" H 13250 8375 50  0001 C CNN
+F 3 "" H 13250 8550 50  0001 C CNN
+F 4 "C191023" H 13250 8550 50  0001 C CNN "LCSC Part"
+	1    13250 8550
+	0    1    1    0
+$EndComp
+Wire Wire Line
+	13250 8400 13250 8250
+$Comp
+L power:GND #PWR08
+U 1 1 63570873
+P 13250 8800
+F 0 "#PWR08" H 13250 8550 50  0001 C CNN
+F 1 "GND" H 13255 8627 50  0000 C CNN
+F 2 "" H 13250 8800 50  0001 C CNN
+F 3 "" H 13250 8800 50  0001 C CNN
+	1    13250 8800
+	1    0    0    -1
+$EndComp
+Wire Wire Line
+	13250 8800 13250 8700
+Wire Wire Line
+	11850 8350 12100 8350
+Wire Wire Line
+	12000 8150 12100 8150
+Wire Wire Line
+	12700 8250 12750 8250
+Wire Wire Line
+	12750 8250 12750 7800
+Wire Wire Line
+	12750 7800 12000 7800
+Wire Wire Line
+	12000 7800 12000 8150
+Connection ~ 12750 8250
+Wire Wire Line
+	12750 8250 12850 8250
 $EndSCHEMATC

Commit message: update gerber files and assembly
Parts:
- removed D5: 1N5819WS, Diode_SMD:D_SOD-323, symbol Diode:1N4148W
- D3: value 1N5819WS -> 1N4148W; footprint Diode_SMD:D_SOD-323 -> Diode_SMD:D_SOD-123; LCSC Part C191023 -> C81598
- R4: LCSC Part (none) -> C23186
- R60: LCSC Part (none) -> C25803
- U15: LCSC Part (none) -> C5613
Connections:
- wire segments 279 -> 277
Changed lines of the file:
@@
 F 2 "Resistor_SMD:R_0603_1608Metric" V 12930 8250 50  0001 C CNN
 F 3 "~" H 13000 8250 50  0001 C CNN
-F 4 "" H 13000 8250 50  0001 C CNN "LCSC Part"
+F 4 "C23186" H 13000 8250 50  0001 C CNN "LCSC Part"
 	1    13000 8250
 	0    -1   -1   0
@@
 P 13250 7900
 F 0 "D3" V 13204 7980 50  0000 L CNN
-F 1 "1N5819WS" V 13295 7980 50  0000 L CNN
-F 2 "Diode_SMD:D_SOD-323" H 13250 7725 50  0001 C CNN
+F 1 "1N4148W" V 13295 7980 50  0000 L CNN
+F 2 "Diode_SMD:D_SOD-123" H 13250 7725 50  0001 C CNN
 F 3 "" H 13250 7900 50  0001 C CNN
-F 4 "C191023" H 13250 7900 50  0001 C CNN "LCSC Part"
+F 4 "C81598" H 13250 7900 50  0001 C CNN "LCSC Part"
 	1    13250 7900
 	0    1    1    0
@@
 F 2 "Package_SO:SOIC-16_3.9x9.9mm_P1.27mm" H 14250 2400 50  0001 C CNN
 F 3 "https://assets.nexperia.com/documents/data-sheet/74HC_HCT165.pdf" H 14250 2400 50  0001 C CNN
+F 4 "C5613" H 14250 2400 50  0001 C CNN "LCSC Part"
 	1    14250 2400
 	1    0    0    -1
@@
 F 2 "Resistor_SMD:R_0603_1608Metric" V 13030 2600 50  0001 C CNN
 F 3 "~" H 13100 2600 50  0001 C CNN
+F 4 "C25803" H 13100 2600 50  0001 C CNN "LCSC Part"
 	1    13100 2600
 	1    0    0    -1
@@
 Wire Notes Line
 	600  8450 600  10450
-$Comp
-L Diode:1N4148W D5
-U 1 1 6355B1F4
-P 13250 8550
-F 0 "D5" V 13204 8630 50  0000 L CNN
-F 1 "1N5819WS" V 13295 8630 50  0000 L CNN
-F 2 "Diode_SMD:D_SOD-323" H 13250 8375 50  0001 C CNN
-F 3 "" H 13250 8550 50  0001 C CNN
-F 4 "C191023" H 13250 8550 50  0001 C CNN "LCSC Part"
-	1    13250 8550
-	0    1    1    0
-$EndComp
-Wire Wire Line
-	13250 8400 13250 8250
-$Comp
-L power:GND #PWR08
-U 1 1 63570873
-P 13250 8800
-F 0 "#PWR08" H 13250 8550 50  0001 C CNN
-F 1 "GND" H 13255 8627 50  0000 C CNN
-F 2 "" H 13250 8800 50  0001 C CNN
-F 3 "" H 13250 8800 50  0001 C CNN
-	1    13250 8800
-	1    0    0    -1
-$EndComp
-Wire Wire Line
-	13250 8800 13250 8700
 Wire Wire Line
 	11850 8350 12100 8350

Commit message: v0.3 submitted to jlcpcb
Parts:
- removed C36: 0.1u, Capacitor_SMD:C_0603_1608Metric, symbol Device:C
- removed R60: 100k, Resistor_SMD:R_0603_1608Metric, symbol Device:R
- removed U15: 74HC165, Package_SO:SOIC-16_3.9x9.9mm_P1.27mm, symbol 74xx:74HC165
- added U15: M24C02-WMN, Package_SO:SOIC-8_3.9x4.9mm_P1.27mm, symbol Memory_EEPROM:M24C02-WMN
Connections:
- net labels added: CARD7_OUT1, CARD7_OUT2, SPI_CS0, SPI_CS1
- net labels removed: ID_CS, SPI_CS
- wire segments 277 -> 260
- no-connect marks 12 -> 14
Other:
- note added: "Board ID in EEPROM\nI2C address 1010{addr2,addr1,addr0}"
- note added: "GPIO for switch control\nI2C address 0100{addr2,addr1,addr0}"
- note removed: "Board ID - can be read in SPI mode 0"
- note removed: "Program control signals"
- moved on the sheet: C13, C37
