File: kicad/as3372/as3372.kicad_pcb (KiCad board)
At the start: 4 copper layers, 80 x 80 mm, 21 parts, among them J1 Conn_01x01, J2 Conn_01x02, J3 Conn_02x20_Odd_Even, U13 LM4040AIM3-2.5, U14 AD5328, U15 M24C02-WMN, U7 PCA9555D

Commit message: daily update
Parts:
- removed U14: AD5328, Package_SO:TSSOP-16_4.4x5mm_P0.65mm
- added C1: 0.1u, Capacitor_SMD:C_0603_1608Metric, F.Cu at (159.8, 91.2)
- added C10: 68n, Capacitor_SMD:C_0603_1608Metric, F.Cu at (225.6, 46.3)
- added C14: 2.2u, Capacitor_SMD:C_1206_3216Metric, F.Cu at (174.0, 52.5)
- added C19: 0.1u, Capacitor_SMD:C_0603_1608Metric, F.Cu at (191.7, 48.8)
- added C2: 0.1u, Capacitor_SMD:C_0603_1608Metric, F.Cu at (168.7, 79.8)
- added C20: 0.1u, Capacitor_SMD:C_0603_1608Metric, F.Cu at (168.2, 67.8)
- added C21: 0.1u, Capacitor_SMD:C_0603_1608Metric, F.Cu at (164.2, 63.3)
- added C22: 0.1u, Capacitor_SMD:C_0603_1608Metric, F.Cu at (193.4, 46.3)
- added C23: 0.1u, Capacitor_SMD:C_0603_1608Metric, F.Cu at (172.3, 70.5)
- added C26: 0.1u, Capacitor_SMD:C_0603_1608Metric, F.Cu at (193.2, 53.9)
- added C28: 0.1u, Capacitor_SMD:C_0603_1608Metric, F.Cu at (179.7, 49.7)
- added C29: 0.1u, Capacitor_SMD:C_0603_1608Metric, F.Cu at (195.7, 48.8)
- added C3: 0.1u, Capacitor_SMD:C_0603_1608Metric, F.Cu at (168.7, 82.3)
- added C30: 0.1u, Capacitor_SMD:C_0603_1608Metric, F.Cu at (172.3, 73.0)
- added C31: 0.1u, Capacitor_SMD:C_0603_1608Metric, F.Cu at (164.2, 73.3)
- added C32: 0.1u, Capacitor_SMD:C_0603_1608Metric, F.Cu at (160.2, 65.8)
- added C33: 0.1u, Capacitor_SMD:C_0603_1608Metric, F.Cu at (195.7, 51.4)
- added C4: 0.1u, Capacitor_SMD:C_0603_1608Metric, F.Cu at (155.8, 91.2)
- added C5: 0.1u, Capacitor_SMD:C_0603_1608Metric, F.Cu at (172.7, 79.8)
- added C6: 0.1u, Capacitor_SMD:C_0603_1608Metric, F.Cu at (151.8, 91.2)
- added C7: 0.1u, Capacitor_SMD:C_0603_1608Metric, F.Cu at (221.6, 46.3)
- added C8: 0.1u, Capacitor_SMD:C_0603_1608Metric, F.Cu at (212.9, 52.9)
- added C9: 68n, Capacitor_SMD:C_0603_1608Metric, F.Cu at (212.9, 55.4)
- added D1: 1N4148, Diode_SMD:D_SOD-123, F.Cu at (180.5, 46.8)
- added R10: 120k, Resistor_SMD:R_0603_1608Metric, F.Cu at (217.6, 46.3)
- added R11: 3.3k, Resistor_SMD:R_0603_1608Metric, F.Cu at (208.8, 55.4)
- added R12: 3.3k, Resistor_SMD:R_0603_1608Metric, F.Cu at (216.9, 52.9)
- added R13: 47k, Resistor_SMD:R_0603_1608Metric, F.Cu at (176.3, 68.0)
- added R14: 20k, Resistor_SMD:R_0603_1608Metric, F.Cu at (176.7, 60.5)
- added R15: 36k, Resistor_SMD:R_0603_1608Metric, F.Cu at (189.2, 58.9)
- added R16: 1k, Resistor_SMD:R_0603_1608Metric, F.Cu at (187.7, 51.4)
- added R17: 1k, Resistor_SMD:R_0603_1608Metric, F.Cu at (164.2, 68.3)
- added R18: 68k, Resistor_SMD:R_0603_1608Metric, F.Cu at (176.7, 58.0)
- added R19: 68k, Resistor_SMD:R_0603_1608Metric, F.Cu at (189.2, 53.9)
- added R21: 1k, Resistor_SMD:R_0603_1608Metric, F.Cu at (180.3, 64.7)
- added R22: 22k, Resistor_SMD:R_0603_1608Metric, F.Cu at (168.2, 70.3)
- added R23: 100k, Resistor_SMD:R_0603_1608Metric, F.Cu at (201.4, 46.3)
- added R24: 100k, Resistor_SMD:R_0603_1608Metric, F.Cu at (176.3, 63.0)
- added R25: 1k, Resistor_SMD:R_0603_1608Metric, F.Cu at (187.7, 48.8)
- added R26: 1k, Resistor_SMD:R_0603_1608Metric, F.Cu at (172.7, 60.5)
- added R27: 10k, Resistor_SMD:R_0603_1608Metric, F.Cu at (173.1, 55.5)
- added R28: 10k, Resistor_SMD:R_0603_1608Metric, F.Cu at (185.4, 46.3)
- added R29: 1k, Resistor_SMD:R_0603_1608Metric, F.Cu at (164.7, 60.3)
- added R30: 47k, Resistor_SMD:R_0603_1608Metric, F.Cu at (164.2, 70.8)
- added R31: 100k, Resistor_SMD:R_0603_1608Metric, F.Cu at (189.4, 46.3)
- added R32: 24k, Resistor_SMD:R_0603_1608Metric, F.Cu at (180.3, 67.2)
- added R33: 1k, Resistor_SMD:R_0603_1608Metric, F.Cu at (178.8, 52.2)
- added R34: 100k, Resistor_SMD:R_0603_1608Metric, F.Cu at (168.2, 62.8)
- added R35: 100k, Resistor_SMD:R_0603_1608Metric, F.Cu at (160.2, 63.3)
- added R36: 56k, Resistor_SMD:R_0603_1608Metric, F.Cu at (172.7, 58.0)
- added R37: 62k, Resistor_SMD:R_0603_1608Metric, F.Cu at (164.2, 65.8)
- added R38: 100k, Resistor_SMD:R_0603_1608Metric, F.Cu at (183.7, 49.7)
- added R39: 100k, Resistor_SMD:R_0603_1608Metric, F.Cu at (168.7, 57.8)
- added R40: 100k, Resistor_SMD:R_0603_1608Metric, F.Cu at (197.4, 46.3)
- added R41: 49.9k, Resistor_SMD:R_0603_1608Metric, F.Cu at (189.2, 56.4)
- added R42: 100k, Resistor_SMD:R_0603_1608Metric, F.Cu at (184.3, 64.7)
- added R43: 100k, Resistor_SMD:R_0603_1608Metric, F.Cu at (176.3, 70.5)
- added R44: 33.2k, Resistor_SMD:R_0603_1608Metric, F.Cu at (180.7, 62.2)
- added R45: 33.2k, Resistor_SMD:R_0603_1608Metric, F.Cu at (160.2, 73.3)
- added R46: 100k, Resistor_SMD:R_0603_1608Metric, F.Cu at (182.8, 52.2)
- added R48: 100k, Resistor_SMD:R_0603_1608Metric, F.Cu at (172.3, 65.5)
- added R49: 49.9k, Resistor_SMD:R_0603_1608Metric, F.Cu at (199.7, 48.8)
- added R5: 2.4k, Resistor_SMD:R_0603_1608Metric, F.Cu at (221.6, 48.8)
- added R50: 100k, Resistor_SMD:R_0603_1608Metric, F.Cu at (160.2, 70.8)
- added R51: 49.9k, Resistor_SMD:R_0603_1608Metric, F.Cu at (184.7, 59.7)
- added R52: 49.9k, Resistor_SMD:R_0603_1608Metric, F.Cu at (168.2, 65.3)
- added R53: 100k, Resistor_SMD:R_0603_1608Metric, F.Cu at (181.2, 54.7)
- added R54: 24.9k, Resistor_SMD:R_0603_1608Metric, F.Cu at (172.3, 68.0)
- added R55: 16.5k, Resistor_SMD:R_0603_1608Metric, F.Cu at (177.2, 55.5)
- added R57: 33.2k, Resistor_SMD:R_0603_1608Metric, F.Cu at (168.2, 72.8)
- added R58: 100k, Resistor_SMD:R_0603_1608Metric, F.Cu at (160.2, 68.3)
- added R59: 10k, Resistor_SMD:R_0603_1608Metric, F.Cu at (164.7, 57.8)
- added R6: 2.4k, Resistor_SMD:R_0603_1608Metric, F.Cu at (208.8, 52.9)
- added R60: 68k, Resistor_SMD:R_0603_1608Metric, F.Cu at (176.3, 65.5)
- added R61: 47k, Resistor_SMD:R_0603_1608Metric, F.Cu at (185.2, 57.2)
- added R62: 1k, Resistor_SMD:R_0603_1608Metric, F.Cu at (191.7, 51.4)
- added R63: 10k, Resistor_SMD:R_0603_1608Metric, F.Cu at (181.2, 57.2)
- added R64: 47k, Resistor_SMD:R_0603_1608Metric, F.Cu at (184.7, 62.2)
- added R65: 33k, Resistor_SMD:R_0603_1608Metric, F.Cu at (168.7, 60.3)
- added R66: 33k, Resistor_SMD:R_0603_1608Metric, F.Cu at (185.2, 54.7)
- added R67: 1k, Resistor_SMD:R_0603_1608Metric, F.Cu at (180.7, 59.7)
- added R68: 1k, Resistor_SMD:R_0603_1608Metric, F.Cu at (172.3, 63.0)
- added R7: 8.2k, Resistor_SMD:R_0603_1608Metric, F.Cu at (217.6, 48.8)
- added R8: 8.2k, Resistor_SMD:R_0603_1608Metric, F.Cu at (220.9, 51.4)
- added R9: 120k, Resistor_SMD:R_0603_1608Metric, F.Cu at (216.9, 55.4)
- added U1: MUX508, Package_SO:SOIC-16_3.9x9.9mm_P1.27mm, F.Cu at (162.4, 84.2)
- added U11: DG442xY, Package_SO:SOIC-16_3.9x9.9mm_P1.27mm, F.Cu at (166.9, 50.8)
- added U17: MUX508, Package_SO:SOIC-16_3.9x9.9mm_P1.27mm, F.Cu at (154.0, 67.8)
- added U19: L79L05_TO92, Package_TO_SOT_THT:TO-92_Inline, F.Cu at (173.1, 48.3)
- added U2: MUX508, Package_SO:SOIC-16_3.9x9.9mm_P1.27mm, F.Cu at (154.0, 84.2)
- added U8: AS3372, Package_SO:SOIC-24W_7.5x15.4mm_P1.27mm, F.Cu at (156.2, 53.5)
- added U9: AD5328, Package_SO:TSSOP-16_4.4x5mm_P0.65mm, F.Cu at (211.2, 48.4)
Connections:
- J3 pad 3: /SPI_MISO -> unconnected-(J3-Pad3)
- J3 pad 6: /SPI_CS1 -> unconnected-(J3-Pad6)
- U7 pad 10: unconnected-(U7-Pad10) -> /VCF_SIG2_CTRL1
- U7 pad 11: unconnected-(U7-Pad11) -> /VCF_SIG2_CTRL2
- U7 pad 13: unconnected-(U7-Pad13) -> /VCF_FM_CTRL
- U7 pad 14: unconnected-(U7-Pad14) -> /VCA_FM_CTRL
- U7 pad 15: unconnected-(U7-Pad15) -> /FILTER_A_CTRL
- U7 pad 16: unconnected-(U7-Pad16) -> /FILTER_B_CTRL
- U7 pad 17: unconnected-(U7-Pad17) -> /FILTER_C_CTRL
- U7 pad 18: unconnected-(U7-Pad18) -> /FILTER_D_CTRL
- U7 pad 20: unconnected-(U7-Pad20) -> /LED_CTRL
- U7 pad 4: unconnected-(U7-Pad4) -> /VCF_SIG1_EN
- U7 pad 5: unconnected-(U7-Pad5) -> /VCF_SIG1_CTRL0
- U7 pad 6: unconnected-(U7-Pad6) -> /VCF_SIG1_CTRL1
- U7 pad 7: /LED_CTRL -> /VCF_SIG1_CTRL2
- U7 pad 8: unconnected-(U7-Pad8) -> /VCF_SIG2_EN
- U7 pad 9: unconnected-(U7-Pad9) -> /VCF_SIG2_CTRL0
Routing:
- net /VCF_SIG1_CTRL2: track 0.00 -> 10.9 mm
- net /LED_CTRL: track 10.9 -> 0.00 mm

Commit message: schematic updates
Parts:
- added C11: 33n, Capacitor_SMD:C_1206_3216Metric, F.Cu at (166.4, 70.9)
- added C12: 33n, Capacitor_SMD:C_1206_3216Metric, F.Cu at (187.8, 49.2)
- added C15: 330p, Capacitor_SMD:C_0805_2012Metric, F.Cu at (185.3, 52.6)
- added C16: 2.2u, Capacitor_SMD:C_1206_3216Metric, F.Cu at (166.4, 67.5)
- added C17: 33n, Capacitor_SMD:C_1206_3216Metric, F.Cu at (172.1, 64.2)
- added C18: 33p, Capacitor_SMD:C_0603_1608Metric, F.Cu at (179.8, 66.6)
- added C27: 2.2u, Capacitor_SMD:C_1206_3216Metric, F.Cu at (187.8, 45.9)
- added C34: 1u, Capacitor_SMD:C_0805_2012Metric, F.Cu at (165.8, 74.1)
- added C35: 1u, Capacitor_SMD:C_0805_2012Metric, F.Cu at (171.5, 67.4)
- added C36: 0.1u, Capacitor_SMD:C_0603_1608Metric, F.Cu at (209.7, 49.6)
- added C38: 4.7u, Capacitor_SMD:C_0805_2012Metric, F.Cu at (165.8, 59.3)
- added C40: 4.7u, Capacitor_SMD:C_0805_2012Metric, F.Cu at (157.4, 77.2)
- added Q1: MMBT3904, Package_TO_SOT_SMD:SOT-23, F.Cu at (179.0, 59.1)
- added Q2: MMBT3904, Package_TO_SOT_SMD:SOT-23, F.Cu at (193.2, 43.1)
- added R1: 100k, Resistor_SMD:R_0402_1005Metric, F.Cu at (159.5, 96.8)
- added R2: 100k, Resistor_SMD:R_0402_1005Metric, F.Cu at (182.0, 82.8)
- added R3: 100k, Resistor_SMD:R_0402_1005Metric, F.Cu at (156.6, 96.8)
- added R4: 100k, Resistor_SMD:R_0402_1005Metric, F.Cu at (162.4, 96.8)
- added R69: 680k, Resistor_SMD:R_0603_1608Metric, F.Cu at (165.6, 76.8)
- added R70: 4k7, Resistor_SMD:R_0603_1608Metric, F.Cu at (201.7, 46.2)
- added R71: 1k, Resistor_SMD:R_0603_1608Metric, F.Cu at (187.8, 69.4)
- added R72: 100k, Resistor_SMD:R_0402_1005Metric, F.Cu at (185.6, 76.2)
- added R73: 22k, Resistor_SMD:R_0603_1608Metric, F.Cu at (205.7, 42.1)
- added TP1: TestPoint, TestPoint:TestPoint_Pad_2.0x2.0mm, F.Cu at (171.3, 70.9)
- added TP10: TestPoint, TestPoint:TestPoint_Pad_2.0x2.0mm, F.Cu at (178.6, 63.3)
- added TP11: TestPoint, TestPoint:TestPoint_Pad_2.0x2.0mm, F.Cu at (189.5, 52.9)
- added TP12: TestPoint, TestPoint:TestPoint_Pad_2.0x2.0mm, F.Cu at (182.6, 63.3)
- added TP13: TestPoint, TestPoint:TestPoint_Pad_2.0x2.0mm, F.Cu at (189.1, 57.0)
- added TP14: TestPoint, TestPoint:TestPoint_Pad_2.0x2.0mm, F.Cu at (227.7, 53.1)
- added TP15: TestPoint, TestPoint:TestPoint_Pad_2.0x2.0mm, F.Cu at (192.7, 47.3)
- added TP2: TestPoint, TestPoint:TestPoint_Pad_2.0x2.0mm, F.Cu at (201.7, 42.9)
- added TP3: TestPoint, TestPoint:TestPoint_Pad_2.0x2.0mm, F.Cu at (175.3, 71.9)
- added TP4: TestPoint, TestPoint:TestPoint_Pad_2.0x2.0mm, F.Cu at (197.7, 46.9)
- added TP5: TestPoint, TestPoint:TestPoint_Pad_2.0x2.0mm, F.Cu at (170.1, 75.0)
- added TP6: TestPoint, TestPoint:TestPoint_Pad_2.0x2.0mm, F.Cu at (197.7, 42.9)
- added TP7: TestPoint, TestPoint:TestPoint_Pad_2.0x2.0mm, F.Cu at (175.8, 67.9)
- added TP8: TestPoint, TestPoint:TestPoint_Pad_2.0x2.0mm, F.Cu at (193.6, 51.4)
- added TP9: TestPoint, TestPoint:TestPoint_Pad_2.0x2.0mm, F.Cu at (185.1, 56.1)
- added U18: NE5532, Package_SO:SOIC-8_3.9x4.9mm_P1.27mm, F.Cu at (159.4, 72.5)
- added U3: NE5532, Package_SO:SOIC-8_3.9x4.9mm_P1.27mm, F.Cu at (176.3, 85.0)
- added U4: TL074, Package_SO:SOIC-14_3.9x8.7mm_P1.27mm, F.Cu at (229.9, 46.0)
- added U5: TL074, Package_SO:SOIC-14_3.9x8.7mm_P1.27mm, F.Cu at (180.8, 46.0)
- added U6: TL074, Package_SO:SOIC-14_3.9x8.7mm_P1.27mm, F.Cu at (172.3, 57.4)
- R23, R24, R31, R34, R35, R36, R38, R39, R40, R42, R43, R44, R45, R46, R48, R50, R53, R54, R55, R57, R58: footprint Resistor_SMD:R_0603_1608Metric -> Resistor_SMD:R_0402_1005Metric
- U7: value PCA9555D -> CAT9555YI-T2
- moved R50 55.1 mm to (212.0, 51.9)
- moved R34 55.1 mm to (220.1, 44.4)
- moved C23 53.6 mm to (217.8, 42.1)
- moved R58 50.9 mm to (209.1, 53.9)
- moved R59 50.2 mm to (213.7, 47.1)
- moved C20 48.8 mm to (209.7, 42.1)
- moved R22 48.8 mm to (209.7, 44.6)
- moved C32 46.7 mm to (205.6, 54.7)
- moved C21 44.5 mm to (205.7, 47.1)
- moved C31 43.4 mm to (201.6, 51.2)
- moved R44 40.6 mm to (217.2, 44.4)
- moved R54 40.2 mm to (209.1, 51.9)
- moved C9 38.4 mm to (248.9, 42.1)
- moved R11 38.4 mm to (244.9, 42.1)
- moved R30 37.9 mm to (197.6, 52.7)
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Connections:
- U11 pad 14: GND -> Net-(R19-Pad1)
- U11 pad 15: GND -> /filter_as3372/WHITE_NOISE
- U11 pad 16: GND -> /WHITE_NOISE_CTRL
- U7 pad 19: unconnected-(U7-Pad19) -> /WHITE_NOISE_CTRL

Commit message: start placing
Parts:
- added C41: 10n, Capacitor_SMD:C_0603_1608Metric, F.Cu at (87.9, 91.0)
- added C42: 10n, Capacitor_SMD:C_0603_1608Metric, F.Cu at (87.9, 89.0)
- added C43: 10n, Capacitor_SMD:C_0603_1608Metric, F.Cu at (86.1, 86.4)
- added C44: 10n, Capacitor_SMD:C_0603_1608Metric, F.Cu at (81.7, 81.8)
- added R74: 15k, Resistor_SMD:R_0603_1608Metric, F.Cu at (84.5, 91.0)
- added R75: 15k, Resistor_SMD:R_0603_1608Metric, F.Cu at (84.5, 89.0)
- added R76: 15k, Resistor_SMD:R_0603_1608Metric, F.Cu at (84.1, 86.4)
- added R77: 15k, Resistor_SMD:R_0603_1608Metric, F.Cu at (81.7, 85.2)
- C10: value 68n -> 8.2p
- C11, C12, C17: footprint Capacitor_SMD:C_1206_3216Metric -> Capacitor_SMD:C_0805_2012Metric
- R10: value 120k -> 20k
- R12: value 3.3k -> 20k
- R41, R49, R51, R52: footprint Resistor_SMD:R_0603_1608Metric -> Resistor_SMD:R_0402_1005Metric
- R6: value 2.4k -> 20k
- R8: value 8.2k -> 20k
- moved R9 172.7 mm to (90.8, 114.2)
- moved C7 172.7 mm to (86.8, 114.2)
- moved C9 172.7 mm to (90.8, 111.7)
- moved R11 172.7 mm to (86.8, 111.7)
- moved C10 172.6 mm to (86.0, 117.9)
- moved U9 169.0 mm to (76.3, 91.8), turned to 180 degrees
- moved R8 168.6 mm to (87.8, 126.8)
- moved R7 168.1 mm to (91.6, 127.4)
- moved R6 166.5 mm to (88.0, 124.6)
- moved TP14 162.9 mm to (69.5, 92.2), turned to 180 degrees
- moved R12 161.6 mm to (86.8, 116.4)
- moved R10 159.8 mm to (87.6, 121.2)
- moved R5 157.6 mm to (99.2, 121.8)
- moved U4 154.8 mm to (93.8, 119.8)
- moved C8 152.4 mm to (99.6, 119.0)
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Connections:
- net /DAC/PAN_VCA_CV_0-5 renamed /DAC/PAN_VCA_CV_DAC
- net /DAC/VCF_CV_0-5 renamed /DAC/VCF_CV_DAC
- net Net-(R65-Pad1) renamed /filter_as3372/VCA6_OUT
- net Net-(R66-Pad1) renamed /filter_as3372/VCA5_OUT
- U7 pad 10: /VCF_SIG2_CTRL1 -> /WHITE_NOISE_CTRL
- U7 pad 11: /VCF_SIG2_CTRL2 -> /LED_CTRL
- U7 pad 13: /VCF_FM_CTRL -> /VCF_SIG1_EN
- U7 pad 14: /VCA_FM_CTRL -> /VCF_SIG1_CTRL0
- U7 pad 15: /FILTER_A_CTRL -> /VCF_SIG1_CTRL1
- U7 pad 16: /FILTER_B_CTRL -> /VCF_SIG1_CTRL2
- U7 pad 17: /FILTER_C_CTRL -> /VCF_SIG2_EN
- U7 pad 18: /FILTER_D_CTRL -> /VCF_SIG2_CTRL0
- U7 pad 19: /WHITE_NOISE_CTRL -> /VCF_SIG2_CTRL1
- U7 pad 20: /LED_CTRL -> /VCF_SIG2_CTRL2
- U7 pad 4: /VCF_SIG1_EN -> /VCF_FM_CTRL
- U7 pad 5: /VCF_SIG1_CTRL0 -> /VCA_FM_CTRL
- U7 pad 6: /VCF_SIG1_CTRL1 -> /FILTER_A_CTRL
- U7 pad 7: /VCF_SIG1_CTRL2 -> /FILTER_B_CTRL
- U7 pad 8: /VCF_SIG2_EN -> /FILTER_C_CTRL
- U7 pad 9: /VCF_SIG2_CTRL0 -> /FILTER_D_CTRL
- U9 pad 4: /DAC/SIG1_VCA1_CV -> /DAC/SIG1_VCA_DAC
- U9 pad 5: /DAC/SIG2_VCA2_CV -> /DAC/SIG2_VCA_DAC
- U9 pad 6: /DAC/MOD_AMOUNT_VCA3_CV -> /DAC/MOD_AMOUNT_VCA3_DAC
- U9 pad 7: /DAC/RESONANCE_CV -> /DAC/RESONANCE_DAC
Routing:
- net /SPI_CS0: track 64.4 -> 0.00 mm
- net /SPI_CLK: track 54.4 -> 0.00 mm
- net /SPI_MOSI: track 54.4 -> 0.00 mm, vias 1 -> 0
- net /I2C_ADDR0: track 33.6 -> 0.00 mm, vias 2 -> 0
- net /SDA1: track 27.8 -> 0.00 mm, vias 2 -> 0
- net /I2C_ADDR1: track 27.5 -> 0.00 mm
- net /SCL1: track 27.4 -> 0.00 mm, vias 1 -> 0
- net /I2C_ADDR2: track 24.3 -> 0.00 mm
- net +5V: track 21.5 -> 0.00 mm, vias 6 -> 0
- net /DAC/VREF_2.5V: track 17.6 -> 0.00 mm
- net GND: track 114.9 -> 97.5 mm, vias 10 -> 0
- net /VCF_SIG1_CTRL2: track 10.9 -> 0.00 mm
- net Net-(J2-Pad1): track 10.5 -> 0.00 mm
- net Net-(D4-Pad1): track 1.89 -> 0.00 mm

Commit message: start placing
Parts:
- added C45: 0.1u, Capacitor_SMD:C_0603_1608Metric, F.Cu at (125.4, 120.0)
- added C46: 0.1u, Capacitor_SMD:C_0603_1608Metric, F.Cu at (115.6, 124.0)
- added U10: TL072, Package_SO:SOIC-8_3.9x4.9mm_P1.27mm, F.Cu at (213.2, 76.1)
- U5: value TL074 -> TL072; footprint Package_SO:SOIC-14_3.9x8.7mm_P1.27mm -> Package_SO:SOIC-8_3.9x4.9mm_P1.27mm
- moved TP15 137.5 mm to (2.80, 145.4), turned to -90 degrees
- moved R70 136.2 mm to (6.20, 141.4), turned to -90 degrees
- moved C40 133.7 mm to (6.00, 145.2), turned to -90 degrees
- moved C38 133.1 mm to (9.60, 140.2), turned to 180 degrees
- moved Q2 130.9 mm to (9.40, 143.4), turned to 180 degrees
- moved R72 129.9 mm to (8.40, 146.4), turned to 0 degrees
- moved R71 128.9 mm to (13.4, 140.0), turned to 0 degrees
- moved C36 126.2 mm to (11.4, 146.4), turned to 180 degrees
- moved Q1 125.7 mm to (13.8, 143.4), turned to 0 degrees
- moved R69 121.9 mm to (15.0, 146.4), turned to 180 degrees
- moved C23 114.4 mm to (218.2, 73.2), turned to -90 degrees
- moved TP10 112.3 mm to (209.4, 70.9)
- moved C33 112.0 mm to (34.9, 142.0), turned to -90 degrees
- moved R60 111.5 mm to (208.2, 74.4), turned to 90 degrees
- moved TP9 111.1 mm to (212.6, 70.5)
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Connections:
- net Net-(R30-Pad1) renamed /filter_as3372/MOD_VCA_OUT
- U11 pad 10: /filter_as3372/VCF_FM -> /filter_as3372/WHITE_NOISE
- U11 pad 11: Net-(U11-Pad11) -> Net-(R19-Pad1)
- U11 pad 14: Net-(R19-Pad1) -> Net-(U11-Pad14)
- U11 pad 15: /filter_as3372/WHITE_NOISE -> /filter_as3372/VCF_FM
- U11 pad 16: /WHITE_NOISE_CTRL -> /VCF_FM_CTRL
- U11 pad 9: /VCF_FM_CTRL -> /WHITE_NOISE_CTRL
- U5 pad 1: Net-(U11-Pad11) -> Net-(U11-Pad7)
- U5 pad 2: Net-(U11-Pad11) -> Net-(U11-Pad7)
- U5 pad 4: +12V -> -12V
- U5 pad 6: Net-(U11-Pad7) -> Net-(U11-Pad14)
- U5 pad 7: Net-(U11-Pad7) -> Net-(U11-Pad14)
- U5 pad 8: /filter_as3372/VCF_OUT_BUFFERED -> +12V

Commit message: start placing
Parts:
- removed H2, H4: MountingHole, MountingHole:MountingHole_3.2mm_M3
- moved TP15 97.9 mm to (88.8, 98.6), turned to 90 degrees
- moved R34 97.5 mm to (122.9, 65.5)
- moved TP10 97.5 mm to (112.5, 59.7)
- moved TP11 97.5 mm to (108.5, 61.3)
- moved R35 97.5 mm to (121.1, 65.1)
- moved TP9 97.5 mm to (115.7, 59.3)
- moved C23 97.5 mm to (121.3, 62.1)
- moved C26 97.5 mm to (111.3, 66.7)
- moved R59 97.5 mm to (109.3, 65.1)
- moved R60 97.5 mm to (111.3, 63.3)
- moved U10 97.5 mm to (116.3, 64.9)
- moved C40 91.8 mm to (85.2, 98.8), turned to 90 degrees
- moved TP6 91.4 mm to (88.3, 49.6)
- moved R72 89.0 mm to (82.8, 97.6), turned to 180 degrees
- moved R70 87.8 mm to (85.0, 102.6), turned to 90 degrees
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