File: kicad/as3372/dac.kicad_sch (KiCad schematic)
At the start: 27 parts, among them U13 LM4040AIM3-2.5, U4 TL074, U9 AD5328

Commit message: updates for v0.2
Parts:
- R5: value 2.4k -> 2k4
- R7: value 8.2k -> 8k2
Connections:
- net GND: no longer U4.5 (+)
- net RESONANCE_CV: now also U4.6 (-), U4.7; no longer C44.1, R77.2
- new net: C44.1, R77.2, U4.5 (+)
Other:
- note added: "Low impedance output for res CV mixing with res modulation source"
- note removed: "Unused"
- moved on the sheet: C41, C42, C43, C44, R74, R75, R76, R77, U4B

Commit message: z3372 v0.2 release to manufacturing
Parts:
- R11: value 3.3k -> 3k3
Connections:
- net MOD_AMOUNT_VCA3_DAC: now also U9.13 (VOUT_H); no longer U9.7 (VOUT_D)
- net RESONANCE_DAC: now also U9.7 (VOUT_D); no longer U9.12 (VOUT_G)

Commit message: mods for v0.3
Parts:
- added C26: 33n, Capacitor_SMD:C_0603_1608Metric, symbol Device:C
- added R16: 20k, Resistor_SMD:R_0603_1608Metric, symbol Device:R
- added R29: 4k3, Resistor_SMD:R_0603_1608Metric, symbol Device:R
- C10: value 8.2p -> 10n; LCSC Part C1685 -> C57112
Connections:
- net GND: now also C26.2, R29.1
- net NOISE_CONTROL_CV: now also C26.1, R16.2, R29.2; no longer U9.6 (VOUT_C)
- new net NOISE_CONTROL_DAC: R16.1, U9.6 (VOUT_C)
Other:
- note added: "Noise Control should be biased to ~0.5V; goes up to 0.85V. RC filter for a lowpass cutoff at <1400 Hz"
- note added: "Pan CVA CV: Take 0V : 5V from DAC shift to -2.5V : 2.5V output 10n cap to give a ~1.6kHz low pass filter"
- note added: "Res CV has an opamp only to provide a low impedance output for res CV mixing with the res modulation source. If res modulation were to be removed this wouldn't be needed."
- note removed: "Low impedance output for res CV mixing with res modulation source"
- note removed: "Pan CVA CV: Take 0V : 5V from DAC shift to -2.5V : 2.5V output 8.2p cap to give a ~1kHz low pass filter"
- moved on the sheet: C10, C44, C9, R10, R11, R12, R5, R6, R7, R77, R8, R9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

Commit message: add proper component part numbers
Parts:
- C26: footprint Capacitor_SMD:C_0603_1608Metric -> Capacitor_SMD:C_0805_2012Metric; LCSC Part C21117 -> C342800
Changed lines of the file:
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@@
     (property "Reference" "C26" (id 0) (at 370.84 111.76 0))
     (property "Value" "33n" (id 1) (at 370.84 114.3 0))
-    (property "Footprint" "Capacitor_SMD:C_0603_1608Metric" (id 2) (at 376.8852 116.84 0)
+    (property "Footprint" "Capacitor_SMD:C_0805_2012Metric" (id 2) (at 376.8852 116.84 0)
       (effects (font (size 1.27 1.27)) hide)
     )
@@
       (effects (font (size 1.27 1.27)) hide)
     )
-    (property "LCSC Part" "C21117" (id 5) (at 375.92 113.03 0)
+    (property "LCSC Part" "C342800" (id 5) (at 375.92 113.03 0)
       (effects (font (size 1.27 1.27)) hide)
     )

Commit message: Zoxnoxious 3372 RTM
Parts:
- C26: value 33n -> 22n; LCSC Part C342800 -> C21122
- R16: value 20k -> 18k; LCSC Part C4184 -> C25810
- R29: value 4k3 -> 9k1; LCSC Part C23159 -> C23260
Other:
- note added: "Noise Control should be biased to ~0.5V; goes up to 1.67V. RC filter for a lowpass cutoff at ~1200 Hz"
- note removed: "Noise Control should be biased to ~0.5V; goes up to 0.85V. RC filter for a lowpass cutoff at <1400 Hz"
Changed lines of the file:
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@@
   (title_block
     (title "Z3372 Signal Processing")
-    (rev "0.2")
+    (rev "0.3")
     (company "Zoxnoxious Engineering")
   )
@@
     (effects (font (size 1.27 1.27)) (justify left bottom))
   )
-  (text "Noise Control should be biased to ~0.5V; goes up to 0.85V.  RC filter\nfor a lowpass cutoff at <1400 Hz"
+  (text "Noise Control should be biased to ~0.5V; goes up to 1.67V.  RC filter\nfor a lowpass cutoff at ~1200 Hz"
     (at 341.63 132.08 0)
     (effects (font (size 1.27 1.27)) (justify left bottom))
@@
     (in_bom yes) (on_board yes)
     (property "Reference" "R16" (id 0) (at 368.3 101.6 90))
-    (property "Value" "20k" (id 1) (at 368.3 106.68 90))
+    (property "Value" "18k" (id 1) (at 368.3 106.68 90))
     (property "Footprint" "Resistor_SMD:R_0603_1608Metric" (id 2) (at 368.3 105.918 90)
       (effects (font (size 1.27 1.27)) hide)
@@
       (effects (font (size 1.27 1.27)) hide)
     )
-    (property "LCSC Part" "C4184" (id 4) (at 368.3 104.14 0)
+    (property "LCSC Part" "C25810" (id 4) (at 368.3 104.14 0)
       (effects (font (size 1.27 1.27)) hide)
     )
@@
     (in_bom yes) (on_board yes)
     (property "Reference" "R29" (id 0) (at 383.54 113.03 90))
-    (property "Value" "4k3" (id 1) (at 388.62 113.03 90))
+    (property "Value" "9k1" (id 1) (at 388.62 113.03 90))
     (property "Footprint" "Resistor_SMD:R_0603_1608Metric" (id 2) (at 387.858 113.03 90)
       (effects (font (size 1.27 1.27)) hide)
@@
       (effects (font (size 1.27 1.27)) hide)
     )
-    (property "LCSC Part" "C23159" (id 4) (at 386.08 113.03 0)
+    (property "LCSC Part" "C23260" (id 4) (at 386.08 113.03 0)
       (effects (font (size 1.27 1.27)) hide)
     )
@@
     (in_bom yes) (on_board yes)
     (property "Reference" "C26" (id 0) (at 370.84 111.76 0))
-    (property "Value" "33n" (id 1) (at 370.84 114.3 0))
+    (property "Value" "22n" (id 1) (at 370.84 114.3 0))
     (property "Footprint" "Capacitor_SMD:C_0805_2012Metric" (id 2) (at 376.8852 116.84 0)
       (effects (font (size 1.27 1.27)) hide)
@@
       (effects (font (size 1.27 1.27)) hide)
     )
-    (property "LCSC Part" "C342800" (id 5) (at 375.92 113.03 0)
-      (effects (font (size 1.27 1.27)) hide)
-    )
+    (property "LCSC Part" "C21122" (id 5) (at 375.92 113.03 0)
+      (effects (font (size 1.27 1.27)) hide)
+    )
