File: kicad/z5524/dac_3394.kicad_sch (KiCad schematic)
At the start: 46 parts, among them U11 DG442xY, U17 AD5328, U18 TL074

Commit message: update LCSC Part numbers, some modification to account for parts
Parts:
- C29, C33: LCSC Part (none) -> C23630
- C65: LCSC Part (none) -> C1588
- R32: LCSC Part (none) -> C22818
- R42: LCSC Part (none) -> C22984
- R46: LCSC Part (none) -> C25805
- R60, R61, R86, R87: LCSC Part (none) -> C25804
- R75, R79: LCSC Part (none) -> C23212
- R76: LCSC Part (none) -> C22935
- R80, R81: LCSC Part (none) -> C4184
- R82: LCSC Part (none) -> C22809
- R89: LCSC Part (none) -> C23196
- R91: LCSC Part (none) -> C31850
- R92: LCSC Part (none) -> C25950
- R95: LCSC Part (none) -> C23153
- R96: LCSC Part (none) -> C23147
- U17: LCSC Part (none) -> C29162
Changed lines of the file:
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@@
+      (effects (font (size 1.27 1.27)) hide)
+    )
+    (property "LCSC Part" "C23212" (at 359.41 50.8 0)
       (effects (font (size 1.27 1.27)) hide)
     )
@@
       (effects (font (size 1.27 1.27)) hide)
     )
+    (property "LCSC Part" "C23196" (at 238.76 121.92 0)
+      (effects (font (size 1.27 1.27)) hide)
+    )
     (pin "1")
     (pin "2")
@@
     )
     (property "Datasheet" "~" (at 354.33 44.45 0)
+      (effects (font (size 1.27 1.27)) hide)
+    )
+    (property "LCSC Part" "C23212" (at 354.33 44.45 0)
       (effects (font (size 1.27 1.27)) hide)
     )
@@
       (effects (font (size 1.27 1.27)) hide)
     )
+    (property "LCSC Part" "C22818" (at 368.3 30.48 0)
+      (effects (font (size 1.27 1.27)) hide)
+    )
     (pin "1")
     (pin "2")
@@
       (effects (font (size 1.27 1.27)) hide)
     )
+    (property "LCSC Part" "C23147" (at 224.79 132.08 0)
+      (effects (font (size 1.27 1.27)) hide)
+    )
     (pin "1")
     (pin "2")
@@
     )
     (property "Datasheet" "https://www.analog.com/en/products/ad5308.html" (at 77.47 57.15 0)
+      (effects (font (size 1.27 1.27)) hide)
+    )
+    (property "LCSC Part" "C29162" (at 77.47 57.15 0)
       (effects (font (size 1.27 1.27)) hide)
     )
@@
     )
     (property "Datasheet" "~" (at 71.12 134.62 0)
+      (effects (font (size 1.27 1.27)) hide)
+    )
+    (property "LCSC Part" "C25804" (at 71.12 134.62 0)
       (effects (font (size 1.27 1.27)) hide)
     )
@@
       (effects (font (size 1.27 1.27)) hide)
     )
+    (property "LCSC Part" "C23153" (at 227.33 143.51 0)
+      (effects (font (size 1.27 1.27)) hide)
+    )
     (pin "1")
     (pin "2")
@@
     )
     (property "Datasheet" "~" (at 204.47 113.03 0)
+      (effects (font (size 1.27 1.27)) hide)
+    )
+    (property "LCSC Part" "C25805" (at 204.47 113.03 0)
       (effects (font (size 1.27 1.27)) hide)
     )
@@
       (effects (font (size 1.27 1.27)) hide)
     )
+    (property "LCSC Part" "C25804" (at 214.63 200.66 0)
+      (effects (font (size 1.27 1.27)) hide)
+    )
     (pin "1")
     (pin "2")
@@
     )
     (property "Datasheet" "~" (at 378.46 50.8 0)
+      (effects (font (size 1.27 1.27)) hide)
+    )
+    (property "LCSC Part" "C22935" (at 378.46 50.8 0)
       (effects (font (size 1.27 1.27)) hide)
     )
@@
       (effects (font (size 1.27 1.27)) hide)
     )
+    (property "LCSC Part" "C22984" (at 226.06 29.21 0)
+      (effects (font (size 1.27 1.27)) hide)
+    )
     (pin "1")
     (pin "2")
@@
     )
     (property "Datasheet" "~" (at 261.62 48.26 0)
+      (effects (font (size 1.27 1.27)) hide)
+    )
+    (property "LCSC Part" "C31850" (at 261.62 48.26 0)
       (effects (font (size 1.27 1.27)) hide)
     )
@@
       (effects (font (size 1.27 1.27)) hide)
     )
+    (property "LCSC Part" "C25804" (at 233.68 185.42 0)
+      (effects (font (size 1.27 1.27)) hide)
+    )
     (pin "1")
     (pin "2")
@@
       (effects (font (size 1.27 1.27)) hide)
     )
+    (property "LCSC Part" "C25804" (at 63.5 128.27 0)
+      (effects (font (size 1.27 1.27)) hide)
+    )
     (pin "1")
     (pin "2")
@@
       (effects (font (size 1.27 1.27)) hide)
     )
+    (property "LCSC Part" "C4184" (at 222.25 207.01 0)
+      (effects (font (size 1.27 1.27)) hide)
+    )
     (pin "1")
     (pin "2")
@@
     )
     (property "Datasheet" "~" (at 194.31 113.03 0)
+      (effects (font (size 1.27 1.27)) hide)
+    )
+    (property "LCSC Part" "C23630" (at 194.31 113.03 0)
       (effects (font (size 1.27 1.27)) hide)
     )
@@
       (effects (font (size 1.27 1.27)) hide)
     )
+    (property "LCSC Part" "C25950" (at 247.65 68.58 0)
+      (effects (font (size 1.27 1.27)) hide)
+    )
     (pin "1")
     (pin "2")
@@
       (effects (font (size 1.27 1.27)) hide)
     )
+    (property "LCSC Part" "C22809" (at 232.41 58.42 0)
+      (effects (font (size 1.27 1.27)) hide)
+    )
     (pin "1")
     (pin "2")
@@
       (effects (font (size 1.27 1.27)) hide)
     )
+    (property "LCSC Part" "C1588" (at 238.76 113.03 0)
+      (effects (font (size 1.27 1.27)) hide)
+    )
     (pin "1")
     (pin "2")
@@
       (effects (font (size 1.27 1.27)) hide)
     )
+    (property "LCSC Part" "C4184" (at 217.17 195.58 0)
+      (effects (font (size 1.27 1.27)) hide)
+    )
     (pin "1")
     (pin "2")
@@
       (effects (font (size 1.27 1.27)) hide)
     )
+    (property "LCSC Part" "C23630" (at 215.9 29.21 0)
+      (effects (font (size 1.27 1.27)) hide)
+    )

Commit message: fix symbol library
Parts:
- U17: symbol Z3340:AD5328 -> z5524:AD5328
Changed lines of the file:
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@@
     )
   )
-  (symbol (lib_id "Z3340:AD5328") (at 77.47 57.15 0) (unit 1)
+  (symbol (lib_id "z5524:AD5328") (at 77.47 57.15 0) (unit 1)
     (in_bom yes) (on_board yes) (dnp no) (fields_autoplaced)
     (property "Reference" "U17" (at 79.4894 43.341 0)
@@
     )
   )
-  (symbol (lib_id "power:-6.5V") (at 378.46 57.15 180) (unit 1)
+  (symbol (lib_id "z5524:-6.5V") (at 378.46 57.15 180) (unit 1)
     (in_bom yes) (on_board yes) (dnp no) (fields_autoplaced)
     (property "Reference" "#PWR048" (at 378.46 59.69 0)
