File: kicad/z3340/as3340.kicad_pcb (KiCad board)
At the start: 4 copper layers, 80 x 80 mm, 153 parts, among them J1 Conn_01x01, J2 Conn_01x02, J3 Conn_02x20_Odd_Even, Q1 2N7002, Q2 2N7002, Q3 MMBT3904, U1 DG442CY+, U10 AS3364, U11 PCA9555D, U12 AD5328, U13 TL074, U14 DG406, U15 M24C02-WMN, U2 AS3340, U3 LM79L05, U4 LM311, U5 TL074, U6 LM4040AIM3-2.5, U7 LM4040B-5, U8 DG442CY+, U9 TL072

Commit message: cleaning up and rename dir to z3340
Parts:
- removed C3: 0.1u, Capacitor_SMD:C_0603_1608Metric
- removed C49: 2u2, Capacitor_THT:C_Rect_L7.2mm_W5.5mm_P5.00mm_FKS2_FKP2_MKS2_MKP2
- added TP8: TestPoint, TestPoint:TestPoint_Pad_2.0x2.0mm, F.Cu at (124.0, 101.2)
- R28: value 1M -> 300k
- R35: value 120k -> 100k
- R37: footprint Resistor_SMD:R_0603_1608Metric -> Resistor_SMD:R_0805_2012Metric
- R62: value 12k -> 100k
- R64: value 82k -> 100k
- moved R62 54.5 mm to (159.8, 86.8)
- moved C42 20.9 mm to (120.1, 131.8), turned to 90 degrees
- moved C4 5.36 mm to (118.2, 78.8), turned to 90 degrees
- moved TP2 2.67 mm to (124.0, 85.0)
- moved C8 2.10 mm to (127.0, 77.8), turned to 0 degrees
- moved R60 1.21 mm to (119.6, 124.1), turned to 180 degrees
- moved C29 1.06 mm to (147.3, 97.6)
- moved Q2 1.06 mm to (151.3, 96.6)
- moved R38 1.06 mm to (147.3, 95.6)
- moved TP6 0.50 mm to (146.1, 100.6)
- moved C31 0.40 mm to (150.0, 92.6)
- moved R31 0.40 mm to (155.5, 92.6)
- moved TP7 0.40 mm to (152.8, 92.6)
- moved U7 0.35 mm to (103.8, 103.0), turned to 90 degrees
- moved C1 0.34 mm to (109.3, 85.3), turned to 90 degrees
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Connections:
- C42 pad 1: Net-(U10C-Iout) -> Net-(U13B--)
- C42 pad 2: Net-(U10D-Iout) -> Net-(C42-Pad2)
- R60 pad 1: Net-(U13B--) -> Net-(C42-Pad2)
- R62 pad 1: /PULSE_VCA_AMOUNT_DAC -> Net-(U4-+)
- R62 pad 2: Net-(U13B--) -> GND
- U10 pad 12: Net-(U10D-Iout) -> Net-(U10C-Iout)
- U10 pad 13: Net-(U10E-Iout) -> Net-(U10C-Iout)
Routing:
- net /PULSE_VCA_AMOUNT_DAC: track 61.0 -> 24.6 mm, vias 3 -> 2
- net Net-(U10E-Iout): track 7.44 -> 0.00 mm
- net Net-(U10D-Iout): track 6.93 -> 0.00 mm
- net Net-(U2-CAP): track 8.23 -> 5.18 mm
- net Net-(C42-Pad2): track 0.00 -> 2.88 mm
- net -5V: track 45.5 -> 42.6 mm
- net Net-(U13B--): track 13.1 -> 10.3 mm
- net Net-(U4-+): track 11.5 -> 13.8 mm
- net Net-(Q1-S): track 3.82 -> 5.57 mm
- net /cem3340/SOFT_SYNC: track 10.5 -> 8.85 mm
- net Net-(U10C-Iout): track 64.6 -> 63.3 mm, vias 3 -> 4
- net Net-(Q2-G): track 9.34 -> 8.58 mm
- net /EXT_MODULATION: track 49.4 -> 50.1 mm
- net +12V: track 43.7 -> 44.4 mm
- net /cem3340/SUMMING_INPUT: track 54.6 -> 54.0 mm
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Other:
- board text added: "TEST POINTS TP1 : HIGH FREQ TRACK TP2 : SOFT SYNC TP3 : VCO SAW TP4 : HARD SYNC TP5 : SYNC COMPARATOR TP6 : VCO TRI TP7 : TRADITIONAL SYNC TP8 : EXTERNAL MOD POST VCA"
- board text added: "Z3340 7/2024 REV 0.8"
- board text removed: "TEST POINTS TP1 : HIGH FREQ TRACK TP2 : SOFT SYNC TP3 : VCO SAW TP4 : HARD SYNC TP5 : SYNC COMPARATOR TP6 : VCO TRI TP7 : TRADITIONAL SYNC"
- board text removed: "Z3340 6/2024 REV 0.7"
