File: kicad/z3340/as3340.kicad_sch (KiCad schematic)
At the start: 42 parts, among them J1 Conn_01x01, J2 Conn_01x02, J3 Conn_02x20_Odd_Even, Q3 MMBT3904, U1 DG442CY+, U10 AS3364, U11 PCA9555D, U13 TL074, U14 DG406, U15 M24C02-WMN, U5 TL074, U8 DG442CY+, U9 TL072

Commit message: cleaning up and rename dir to z3340
Parts:
- added TP8: TestPoint, TestPoint:TestPoint_Pad_2.0x2.0mm, symbol Connector:TestPoint
Connections:
- net EXT_MOD_SCALED: now also TP8.1
Other:
- moved on the sheet: C12, C13, C19, C21, C27, C37, C38, C45, C47, C9, J1, J2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
