File: kicad/z3340/output_mix.kicad_sch (KiCad schematic)
At the start: 26 parts, among them U10 AS3364, U13 TL074, U8 DG442CY+, U9 TL072

Commit message: cleaning up and rename dir to z3340
Parts:
- removed C49: 2u2, Capacitor_THT:C_Rect_L7.2mm_W5.5mm_P5.00mm_FKS2_FKP2_MKS2_MKP2, symbol Device:C
- removed R62: 12k, Resistor_SMD:R_0603_1608Metric, symbol Device:R
- R35: value 120k -> 100k; LCSC Part C25808 -> C25803
- R64: value 82k -> 100k; LCSC Part C23254 -> C25803
Connections:
- net at C41.2, R61.1, U10.5 (Iout)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: now also U10.12 (Iout), U10.13 (Iout); no longer C42.1
- net at R59.2, U13.6 (-): now also C42.1; no longer R60.1
- net at C42.2: now also R60.1; no longer U10.12 (Iout)
Other:
- note added: "Output One and Two Scaling: One has VCA controlled output levels that are AC coupled. Output Two fixed levels between Pulse and Saw and unipolar."
- note removed: "91k may be preferred"
- note removed: "Impedance from DAC ~12k"
- note removed: "Outpus One and Two Scaling: One has VCA controlled output levels that are AC coupled (tri / saw) or at least offset (pulse). No AC coupling on the pulse to keep it looking sharp for modulation. Output Two fixed levels between Pulse and Saw and unipolar."
- moved on the sheet: C41, C42, R22, R60, R61, U13C

Commit message: cleanup references after file renaming
Parts:
- U10: symbol as3340:AS3364 -> z3340:AS3364
Changed lines of the file:
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@@
     )
   )
-  (symbol (lib_id "as3340:AS3364") (at 96.52 40.64 0) (unit 4)
+  (symbol (lib_id "z3340:AS3364") (at 96.52 40.64 0) (unit 4)
     (in_bom yes) (on_board yes) (dnp no) (fields_autoplaced)
     (property "Reference" "U10" (at 97.155 47.3893 0)
@@
     )
   )
-  (symbol (lib_id "as3340:AS3364") (at 95.25 63.5 0) (unit 3)
+  (symbol (lib_id "z3340:AS3364") (at 95.25 63.5 0) (unit 3)
     (in_bom yes) (on_board yes) (dnp no) (fields_autoplaced)
     (property "Reference" "U10" (at 97.155 70.2493 0)
@@
     )
   )
-  (symbol (lib_id "as3340:AS3364") (at 64.77 217.17 0) (unit 2)
+  (symbol (lib_id "z3340:AS3364") (at 64.77 217.17 0) (unit 2)
     (in_bom yes) (on_board yes) (dnp no) (fields_autoplaced)
     (property "Reference" "U10" (at 66.675 223.9193 0)
@@
     )
   )
-  (symbol (lib_id "as3340:AS3364") (at 95.25 86.36 0) (unit 5)
+  (symbol (lib_id "z3340:AS3364") (at 95.25 86.36 0) (unit 5)
     (in_bom yes) (on_board yes) (dnp no)
     (property "Reference" "U10" (at 97.155 93.1093 0)

Commit message: updates for v0.9: polygons, LED resistor, mod amount
Parts:
- C39, C41: LCSC (none) -> C1653; LCSC Part C1653 -> (none)
- R22, R50: LCSC (none) -> C22807; LCSC Part C22807 -> (none)
- R23, R24, R29, R53, R55, R56, R59, R60, R61: LCSC (none) -> C25819; LCSC Part C25819 -> (none)
- R35, R49, R54, R64: LCSC (none) -> C25803; LCSC Part C25803 -> (none)
- R52, R63: LCSC (none) -> C17738; LCSC Part C17738 -> (none)
- U13: LCSC (none) -> C96507; LCSC Part C96507 -> (none)
- U8: LCSC (none) -> C2673321; LCSC Part C2673321 -> (none)
- U9: LCSC (none) -> C6961; LCSC Part C6961 -> (none)
Changed lines of the file:
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@@
   (title_block
     (title "Zoxnoxious 3340 Oscillator")
-    (date "2024-07-15")
-    (rev "0.8")
+    (date "2025-02-06")
+    (rev "0.9")
     (company "Zoxnoxious Engineering")
   )
@@
       (effects (font (size 1.27 1.27)) hide)
     )
-    (property "LCSC Part" "C25803" (at 78.74 63.5 0)
+    (property "LCSC" "C25803" (at 78.74 63.5 0)
       (effects (font (size 1.27 1.27)) hide)
     )
@@
       (effects (font (size 1.27 1.27)) hide)
     )
-    (property "LCSC Part" "C22807" (at 116.84 133.35 0)
+    (property "LCSC" "C22807" (at 116.84 133.35 0)
       (effects (font (size 1.27 1.27)) hide)
     )
@@
       (effects (font (size 1.27 1.27)) hide)
     )
-    (property "LCSC Part" "C2673321" (at 102.87 133.35 0)
+    (property "LCSC" "C2673321" (at 102.87 133.35 0)
       (effects (font (size 1.27 1.27)) hide)
     )
@@
       (effects (font (size 1.27 1.27)) hide)
     )
-    (property "LCSC Part" "C2673321" (at 102.87 152.4 0)
+    (property "LCSC" "C2673321" (at 102.87 152.4 0)
       (effects (font (size 1.27 1.27)) hide)
     )
@@
       (effects (font (size 1.27 1.27)) hide)
     )
-    (property "LCSC Part" "C96507" (at 142.24 88.9 0)
+    (property "LCSC" "C96507" (at 142.24 88.9 0)
       (effects (font (size 1.27 1.27)) hide)
     )
@@
       (effects (font (size 1.27 1.27)) hide)
     )
-    (property "LCSC Part" "C96507" (at 191.77 91.44 0)
+    (property "LCSC" "C96507" (at 191.77 91.44 0)
       (effects (font (size 1.27 1.27)) hide)
     )
@@
       (effects (font (size 1.27 1.27)) hide)
     )
-    (property "LCSC Part" "C25803" (at 78.74 86.36 0)
+    (property "LCSC" "C25803" (at 78.74 86.36 0)
       (effects (font (size 1.27 1.27)) hide)
     )
@@
       (effects (font (size 1.27 1.27)) hide)
     )
-    (property "LCSC Part" "C17738" (at 210.82 138.43 0)
+    (property "LCSC" "C17738" (at 210.82 138.43 0)
       (effects (font (size 1.27 1.27)) hide)
     )
@@
       (effects (font (size 1.27 1.27)) hide)
     )
-    (property "LCSC Part" "C25819" (at 78.74 40.64 0)
+    (property "LCSC" "C25819" (at 78.74 40.64 0)
       (effects (font (size 1.27 1.27)) hide)
     )
@@
       (effects (font (size 1.27 1.27)) hide)
     )
-    (property "LCSC Part" "C25803" (at 123.19 160.02 0)
+    (property "LCSC" "C25803" (at 123.19 160.02 0)
       (effects (font (size 1.27 1.27)) hide)
     )
@@
       (effects (font (size 1.27 1.27)) hide)
     )
-    (property "LCSC Part" "C25819" (at 140.97 78.74 0)
+    (property "LCSC" "C25819" (at 140.97 78.74 0)
       (effects (font (size 1.27 1.27)) hide)
     )
@@
       (effects (font (size 1.27 1.27)) hide)
     )
-    (property "LCSC Part" "C25803" (at 116.84 152.4 0)
+    (property "LCSC" "C25803" (at 116.84 152.4 0)
       (effects (font (size 1.27 1.27)) hide)
     )
@@
       (effects (font (size 1.27 1.27)) hide)
     )
-    (property "LCSC Part" "C25819" (at 191.77 80.01 0)
+    (property "LCSC" "C25819" (at 191.77 80.01 0)
       (effects (font (size 1.27 1.27)) hide)
     )
@@
       (effects (font (size 1.27 1.27)) hide)
     )
-    (property "LCSC Part" "C25819" (at 161.29 88.9 0)
+    (property "LCSC" "C25819" (at 161.29 88.9 0)
       (effects (font (size 1.27 1.27)) hide)
     )
@@
       (effects (font (size 1.27 1.27)) hide)
     )
-    (property "LCSC Part" "C17738" (at 209.55 91.44 0)
+    (property "LCSC" "C17738" (at 209.55 91.44 0)
       (effects (font (size 1.27 1.27)) hide)
     )
@@
       (effects (font (size 1.27 1.27)) hide)
     )
-    (property "LCSC Part" "C1653" (at 140.97 71.12 90)
+    (property "LCSC" "C1653" (at 140.97 71.12 90)
       (effects (font (size 1.27 1.27)) hide)
     )
@@
       (effects (font (size 1.27 1.27)) hide)
     )
-    (property "LCSC Part" "C96507" (at 151.13 135.89 0)
+    (property "LCSC" "C96507" (at 151.13 135.89 0)
       (effects (font (size 1.27 1.27)) hide)
     )
@@
       (effects (font (size 1.27 1.27)) hide)
     )
-    (property "LCSC Part" "C25819" (at 149.86 123.19 0)
+    (property "LCSC" "C25819" (at 149.86 123.19 0)
       (effects (font (size 1.27 1.27)) hide)
     )
@@
       (effects (font (size 1.27 1.27)) hide)
     )
-    (property "LCSC Part" "C25819" (at 193.04 127 0)
+    (property "LCSC" "C25819" (at 193.04 127 0)
       (effects (font (size 1.27 1.27)) hide)
     )
@@
       (effects (font (size 1.27 1.27)) hide)
     )
-    (property "LCSC Part" "C25819" (at 171.45 135.89 0)
+    (property "LCSC" "C25819" (at 171.45 135.89 0)
       (effects (font (size 1.27 1.27)) hide)
     )
@@
       (effects (font (size 1.27 1.27)) hide)
     )
-    (property "LCSC Part" "C96507" (at 193.04 138.43 0)
+    (property "LCSC" "C96507" (at 193.04 138.43 0)
       (effects (font (size 1.27 1.27)) hide)
     )
@@
       (effects (font (size 1.27 1.27)) hide)
     )
-    (property "LCSC Part" "C1653" (at 149.86 114.3 90)
+    (property "LCSC" "C1653" (at 149.86 114.3 90)
       (effects (font (size 1.27 1.27)) hide)
     )
@@
       (effects (font (size 1.27 1.27)) hide)
     )
-    (property "LCSC Part" "C22807" (at 45.72 69.85 0)
+    (property "LCSC" "C22807" (at 45.72 69.85 0)
       (effects (font (size 1.27 1.27)) hide)
     )
@@
       (effects (font (size 1.27 1.27)) hide)
     )
-    (property "LCSC Part" "C25819" (at 50.8 217.17 0)
+    (property "LCSC" "C25819" (at 50.8 217.17 0)
       (effects (font (size 1.27 1.27)) hide)
     )
@@
       (effects (font (size 1.27 1.27)) hide)
     )
-    (property "LCSC Part" "C25819" (at 99.06 208.28 0)
+    (property "LCSC" "C25819" (at 99.06 208.28 0)
       (effects (font (size 1.27 1.27)) hide)
     )
@@
       (effects (font (size 1.27 1.27)) hide)
     )
-    (property "LCSC Part" "" (at 171.45 88.9 90)
+    (property "LCSC" "" (at 171.45 88.9 90)
       (effects (font (size 1.27 1.27)) hide)
     )
@@
       (effects (font (size 1.27 1.27)) hide)
     )
-    (property "LCSC Part" "C6961" (at 100.33 219.71 0)
-      (effects (font (size 1.27 1.27)) hide)
-    )
+    (property "LCSC" "C6961" (at 100.33 219.71 0)
+      (effects (font (size 1.27 1.27)) hide)
+    )

Commit message: updates to z3340 and poledancer schematics and layout
Parts:
- R23: value 47k -> 39k; LCSC C25819 -> C23153
- R64: value 100k -> 82k; LCSC C25803 -> C23254
Changed lines of the file:
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@@
       (effects (font (size 1.27 1.27)))
     )
-    (property "Value" "100k" (at 78.74 88.9 90)
+    (property "Value" "82k" (at 78.74 88.9 90)
       (effects (font (size 1.27 1.27)))
     )
@@
       (effects (font (size 1.27 1.27)) hide)
     )
-    (property "LCSC" "C25803" (at 78.74 86.36 0)
+    (property "LCSC" "C23254" (at 78.74 86.36 0)
       (effects (font (size 1.27 1.27)) hide)
     )
@@
       (effects (font (size 1.27 1.27)))
     )
-    (property "Value" "47k" (at 78.74 43.18 90)
+    (property "Value" "39k" (at 78.74 43.18 90)
       (effects (font (size 1.27 1.27)))
     )
@@
       (effects (font (size 1.27 1.27)) hide)
     )
-    (property "LCSC" "C25819" (at 78.74 40.64 0)
+    (property "LCSC" "C23153" (at 78.74 40.64 0)
       (effects (font (size 1.27 1.27)) hide)
     )
