File: kicad/z3340/z3340.kicad_pcb (KiCad board)
At the start: 4 copper layers, 80 x 80 mm, 152 parts, among them J1 Conn_01x01, J2 Conn_01x02, J3 Conn_02x20_Odd_Even, Q1 2N7002, Q2 2N7002, Q3 MMBT3904, U1 DG442CY+, U10 AS3364, U11 PCA9555D, U12 AD5328, U13 TL074, U14 DG406, U15 M24C02-WMN, U2 AS3340, U3 LM79L05, U4 LM311, U5 TL074, U6 LM4040AIM3-2.5, U7 LM4040B-5, U8 DG442CY+, U9 TL072

Commit message: updates to z3340 and poledancer schematics and layout
Changed lines of the file:
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@@
     (property "ki_keywords" "cap capacitor")
     (attr smd)
-    (fp_text reference "C8" (at -0.75 -1.75) (layer "F.SilkS")
+    (fp_text reference "C8" (at 0 2.05) (layer "F.SilkS")
         (effects (font (size 1 1) (thickness 0.15)))
     )
