File: kicad/z3372/dac.kicad_sch (KiCad schematic)
At the start: 27 parts, among them U12 AD5328, U5 TL074

Commit message: z3372 updated ready for RTM
Parts:
- C12, C24, C28, C4, C40: LCSC (none) -> C14663; LCSC Part C14663 -> (none)
- C22: LCSC (none) -> C21122; LCSC Part C21122 -> (none)
- C27: LCSC (none) -> C1622; LCSC Part C1622 -> (none)
- C41, C42, C7: LCSC (none) -> C57112; LCSC Part C57112 -> (none)
- C44: LCSC (none) -> C1779; LCSC Part C1779 -> (none)
- R12: LCSC (none) -> C25819; LCSC Part C25819 -> (none)
- R13, R7: LCSC (none) -> C23260; LCSC Part C23260 -> (none)
- R29, R5, R51, R54: LCSC (none) -> C22809; LCSC Part C22809 -> (none)
- R31, R33, R34, R37, R40, R41: LCSC (none) -> C4184; LCSC Part C4184 -> (none)
- R36: LCSC (none) -> C4216; LCSC Part C4216 -> (none)
- U12: LCSC (none) -> C29162; LCSC Part C29162 -> (none)
- U5: LCSC (none) -> C96507; LCSC Part C96507 -> (none)
Changed lines of the file:
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@@
   (title_block
     (title "Z3372 Signal Processor")
-    (date "2025-02-02")
+    (date "2025-02-03")
     (rev "0.5")
     (company "Zoxnoxious Engineering")
@@
       (effects (font (size 1.27 1.27)) hide)
     )
-    (property "LCSC Part" "C1779" (at 85.09 33.02 0)
+    (property "LCSC" "C1779" (at 85.09 33.02 0)
       (effects (font (size 1.27 1.27)) hide)
     )
@@
       (effects (font (size 1.27 1.27)) hide)
     )
-    (property "LCSC Part" "C14663" (at 85.09 39.37 0)
+    (property "LCSC" "C14663" (at 85.09 39.37 0)
       (effects (font (size 1.27 1.27)) hide)
     )
@@
       (effects (font (size 1.27 1.27)) hide)
     )
-    (property "LCSC Part" "C14663" (at 55.88 227.33 0)
+    (property "LCSC" "C14663" (at 55.88 227.33 0)
       (effects (font (size 1.27 1.27)) hide)
     )
@@
       (effects (font (size 1.27 1.27)) hide)
     )
-    (property "LCSC Part" "C22809" (at 209.55 38.1 0)
+    (property "LCSC" "C22809" (at 209.55 38.1 0)
       (effects (font (size 1.27 1.27)) hide)
     )
@@
       (effects (font (size 1.27 1.27)) hide)
     )
-    (property "LCSC Part" "C96507" (at 49.53 237.49 0)
+    (property "LCSC" "C96507" (at 49.53 237.49 0)
       (effects (font (size 1.27 1.27)) hide)
     )
@@
       (effects (font (size 1.27 1.27)) hide)
     )
-    (property "LCSC Part" "C22809" (at 208.28 130.81 0)
+    (property "LCSC" "C22809" (at 208.28 130.81 0)
       (effects (font (size 1.27 1.27)) hide)
     )
@@
       (effects (font (size 1.27 1.27)) hide)
     )
-    (property "LCSC Part" "C29162" (at 76.2 57.15 0)
+    (property "LCSC" "C29162" (at 76.2 57.15 0)
       (effects (font (size 1.27 1.27)) hide)
     )
@@
       (effects (font (size 1.27 1.27)) hide)
     )
-    (property "LCSC Part" "C23260" (at 217.17 139.7 0)
+    (property "LCSC" "C23260" (at 217.17 139.7 0)
       (effects (font (size 1.27 1.27)) hide)
     )
@@
       (effects (font (size 1.27 1.27)) hide)
     )
-    (property "LCSC Part" "C22809" (at 208.28 110.49 0)
+    (property "LCSC" "C22809" (at 208.28 110.49 0)
       (effects (font (size 1.27 1.27)) hide)
     )
@@
       (effects (font (size 1.27 1.27)) hide)
     )
-    (property "LCSC Part" "C25819" (at 314.96 45.72 0)
+    (property "LCSC" "C25819" (at 314.96 45.72 0)
       (effects (font (size 1.27 1.27)) hide)
     )
@@
       (effects (font (size 1.27 1.27)) hide)
     )
-    (property "LCSC Part" "C4184" (at 314.96 92.71 0)
+    (property "LCSC" "C4184" (at 314.96 92.71 0)
       (effects (font (size 1.27 1.27)) hide)
     )
@@
       (effects (font (size 1.27 1.27)) hide)
     )
-    (property "LCSC Part" "C14663" (at 226.06 116.84 0)
+    (property "LCSC" "C14663" (at 226.06 116.84 0)
       (effects (font (size 1.27 1.27)) hide)
     )
@@
       (effects (font (size 1.27 1.27)) hide)
     )
-    (property "LCSC Part" "C57112" (at 218.44 62.23 0)
+    (property "LCSC" "C57112" (at 218.44 62.23 0)
       (effects (font (size 1.27 1.27)) hide)
     )
@@
       (effects (font (size 1.27 1.27)) hide)
     )
-    (property "LCSC Part" "C96507" (at 396.24 200.66 0)
+    (property "LCSC" "C96507" (at 396.24 200.66 0)
       (effects (font (size 1.27 1.27)) hide)
     )
@@
       (effects (font (size 1.27 1.27)) hide)
     )
-    (property "LCSC Part" "C4184" (at 306.07 86.36 0)
+    (property "LCSC" "C4184" (at 306.07 86.36 0)
       (effects (font (size 1.27 1.27)) hide)
     )
@@
       (effects (font (size 1.27 1.27)) hide)
     )
-    (property "LCSC Part" "C4184" (at 316.23 133.35 0)
+    (property "LCSC" "C4184" (at 316.23 133.35 0)
       (effects (font (size 1.27 1.27)) hide)
     )
@@
       (effects (font (size 1.27 1.27)) hide)
     )
-    (property "LCSC Part" "C96507" (at 332.74 83.82 0)
+    (property "LCSC" "C96507" (at 332.74 83.82 0)
       (effects (font (size 1.27 1.27)) hide)
     )
@@
       (effects (font (size 1.27 1.27)) hide)
     )
-    (property "LCSC Part" "C96507" (at 332.74 135.89 0)
+    (property "LCSC" "C96507" (at 332.74 135.89 0)
       (effects (font (size 1.27 1.27)) hide)
     )
@@
       (effects (font (size 1.27 1.27)) hide)
     )
-    (property "LCSC Part" "C4184" (at 332.74 124.46 0)
+    (property "LCSC" "C4184" (at 332.74 124.46 0)
       (effects (font (size 1.27 1.27)) hide)
     )
@@
       (effects (font (size 1.27 1.27)) hide)
     )
-    (property "LCSC Part" "C21122" (at 332.74 114.3 0)
+    (property "LCSC" "C21122" (at 332.74 114.3 0)
       (effects (font (size 1.27 1.27)) hide)
     )
@@
       (effects (font (size 1.27 1.27)) hide)
     )
-    (property "LCSC Part" "C1622" (at 320.04 92.71 0)
+    (property "LCSC" "C1622" (at 320.04 92.71 0)
       (effects (font (size 1.27 1.27)) hide)
     )
@@
       (effects (font (size 1.27 1.27)) hide)
     )
-    (property "LCSC Part" "C4184" (at 330.2 72.39 0)
+    (property "LCSC" "C4184" (at 330.2 72.39 0)
       (effects (font (size 1.27 1.27)) hide)
     )
@@
       (effects (font (size 1.27 1.27)) hide)
     )
-    (property "LCSC Part" "C22809" (at 209.55 58.42 0)
+    (property "LCSC" "C22809" (at 209.55 58.42 0)
       (effects (font (size 1.27 1.27)) hide)
     )
@@
       (effects (font (size 1.27 1.27)) hide)
     )
-    (property "LCSC Part" "C14663" (at 55.88 248.92 0)
+    (property "LCSC" "C14663" (at 55.88 248.92 0)
       (effects (font (size 1.27 1.27)) hide)
     )
@@
       (effects (font (size 1.27 1.27)) hide)
     )
-    (property "LCSC Part" "C4216" (at 331.47 36.83 0)
+    (property "LCSC" "C4216" (at 331.47 36.83 0)
       (effects (font (size 1.27 1.27)) hide)
     )
@@
       (effects (font (size 1.27 1.27)) hide)
     )
-    (property "LCSC Part" "C57112" (at 331.47 26.67 0)
+    (property "LCSC" "C57112" (at 331.47 26.67 0)
       (effects (font (size 1.27 1.27)) hide)
     )
@@
       (effects (font (size 1.27 1.27)) hide)
     )
-    (property "LCSC Part" "C4184" (at 306.07 81.28 0)
+    (property "LCSC" "C4184" (at 306.07 81.28 0)
       (effects (font (size 1.27 1.27)) hide)
     )
@@
       (effects (font (size 1.27 1.27)) hide)
     )
-    (property "LCSC Part" "C23260" (at 218.44 116.84 0)
+    (property "LCSC" "C23260" (at 218.44 116.84 0)
       (effects (font (size 1.27 1.27)) hide)
     )
@@
       (effects (font (size 1.27 1.27)) hide)
     )
-    (property "LCSC Part" "C57112" (at 218.44 41.91 0)
+    (property "LCSC" "C57112" (at 218.44 41.91 0)
       (effects (font (size 1.27 1.27)) hide)
     )
@@
       (effects (font (size 1.27 1.27)) hide)
     )
-    (property "LCSC Part" "C14663" (at 226.06 139.7 0)
+    (property "LCSC" "C14663" (at 226.06 139.7 0)
       (effects (font (size 1.27 1.27)) hide)
     )
@@
       (effects (font (size 1.27 1.27)) hide)
     )
-    (property "LCSC Part" "C96507" (at 332.74 48.26 0)
-      (effects (font (size 1.27 1.27)) hide)
-    )
+    (property "LCSC" "C96507" (at 332.74 48.26 0)
+      (effects (font (size 1.27 1.27)) hide)
+    )
