File: kicad/vca_backplane/output_select.kicad_sch (KiCad schematic)
At the start: 60 parts, among them J10 AudioJack3DPDT, J9 AudioJack3DPDT, U10 NE5532, U12 MAX333A, U13 MAX333A, U14 NE5532, U4 MCP4822, U5 PCA9555PW, U7 AS3360, U9 PS508

Commit message: fix some poor routing
Parts:
- removed C?: 47u, Capacitor_THT:CP_Radial_D6.3mm_P2.50mm, symbol Device:C
- added C28: 47u, Capacitor_THT:CP_Radial_D6.3mm_P2.50mm, symbol Device:C_Polarized
- C27: renamed from C?; value C_Polarized -> 47u; footprint (none) -> Capacitor_THT:CP_Radial_D6.3mm_P2.50mm; Digikey (none) -> 493-4538-2-ND
- R23, R25: renamed from R?; value R -> 2k; footprint (none) -> Resistor_SMD:R_0603_1608Metric
Connections:
- net GND: now also C26.1, C4.2, R23.2, R25.2, RV1.1, RV1.4; no longer C26.2, C4.1, RV1.3, RV1.6
- net at U7.6 (Signal): now also C27.2
- net at U7.9 (Signal): now also C28.2
- net at R10.1, TP14.1: now also C26.2, RV1.3; no longer C26.1, RV1.1
- net at R4.1, TP13.1: now also C4.1, RV1.6; no longer C4.2, RV1.4
- net at R25.1, U12.13: now also C28.1
- net at U12.8: now also C27.1, R23.1
Other:
- note added: "AC Coupled via 47u polymer AL cap and 2k resistor"
- note added: "DECOUPING CAPS"
- moved on the sheet: C10, C13, C14, C22, C24, C26, C27, C4, C9, R10, R12, R13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

Commit message: getting to v0.2 for backplane
Parts:
- removed R24: DNP, Resistor_THT:R_Axial_DIN0207_L6.3mm_D2.5mm_P10.16mm_Horizontal, symbol Device:R
- R10, R4: value 12k -> 10k; LCSC Part C22790 -> (none)
- R23, R25: footprint Resistor_SMD:R_0603_1608Metric -> Resistor_SMD:R_1206_3216Metric; LCSC Part (none) -> C17944
Other:
- moved on the sheet: C20, R16

Commit message: v0.2 of backplane submitted to jlcpcb
Parts:
- C10: LCSC (none) -> C1779; LCSC Part C1779 -> (none)
- C13, C14, C15, C16, C17, C18, C22, C23, C24, C25, C26, C4, C6, C7, C8, C9: LCSC (none) -> C14663; LCSC Part C14663 -> (none)
- C19, C20: LCSC (none) -> C14858; LCSC Part C14858 -> (none)
- C21: LCSC (none) -> C1664; LCSC Part C1664 -> (none)
- C27, C28: Digikey 493-4538-2-ND -> 493-10780-1-ND
- C5: LCSC (none) -> C53987; LCSC Part C53987 -> (none)
- D1: LCSC (none) -> C2286; LCSC Part C2286 -> (none)
- R10, R4: LCSC (none) -> C25804
- R11: LCSC (none) -> C22975; LCSC Part C22975 -> (none)
- R12, R13, R14, R5, R7, R8, R9: LCSC (none) -> C25819; LCSC Part C25819 -> (none)
- R15, R16: LCSC (none) -> C17713; LCSC Part C17713 -> (none)
- R17, R18: LCSC (none) -> C25804; LCSC Part C25804 -> (none)
- R19, R20, R22: LCSC (none) -> C17887; LCSC Part C17887 -> (none)
- R21: LCSC (none) -> C23186; LCSC Part C23186 -> (none)
- R23, R25: LCSC (none) -> C17944; LCSC Part C17944 -> (none)
- U10, U14: LCSC (none) -> C7426; LCSC Part C7426 -> (none)
- U4: LCSC (none) -> C16040; LCSC Part C16040 -> (none)
- U5: LCSC (none) -> C83265; LCSC Part C83265 -> (none)
Other:
- note added: "AC Coupled via 47u decent electro cap and 2k resistor"
- note removed: "AC Coupled via 47u polymer AL cap and 2k resistor"
- company: (none) -> Zoxnoxious Engineering
- title: (none) -> Zoxnoxious Backplane and VCA

Commit message: updates to 0.4 as3340 and 0.3 backplane
Connections:
- net MIX2_A0: now also U5.18 (IO1_5); no longer U5.20 (IO1_7)
- net MIX2_A1: now also U5.19 (IO1_6); no longer U5.13 (IO1_0)
- net MIX2_A2: now also U5.20 (IO1_7); no longer U5.14 (IO1_1)
- net MIX2_SELECTED: now also TP12.1
- net MIX2_SELECT_EN: now also U5.17 (IO1_4); no longer U5.19 (IO1_6)
- net MIX2_VCA_IN: no longer TP12.1
- net at R11.2: now also U5.13 (IO1_0); no longer U5.15 (IO1_2)
Other:
- moved on the sheet: D1, R11, R8, TP12

Commit message: schematic for backplane v0.3: change Pi GPIOs for SPI; switch output jacks; add external input
Parts:
- removed C21: 330p, Capacitor_SMD:C_0603_1608Metric, symbol Device:C
- removed C24, C25: 0.1u, Capacitor_SMD:C_0603_1608Metric, symbol Device:C
- removed J10, J9: AudioJack3DPDT, Connector_Audio:Jack_6.35mm_CUI_SJ_63043F, symbol vca_backplane:AudioJack3DPDT
- removed R8: 47k, Resistor_SMD:R_0603_1608Metric, symbol Device:R
- removed TP12: TestPoint, TestPoint:TestPoint_Pad_2.0x2.0mm, symbol Connector:TestPoint
- removed unit 2 of U10
- removed U12, U13: MAX333A, Package_SO:SOIC-20W_7.5x12.8mm_P1.27mm, symbol Analog_Switch:MAX333A
- removed unit 2 of U14
- removed unit 3 of U14
- removed U9: PS508, Package_SO:SOIC-16_3.9x9.9mm_P1.27mm, symbol vca_backplane:MAX308
- added J13, J9: AudioJack_729JH, project_footprints:Jack_3.5mm_729JH-R_Horizontal, symbol vca_backplane:AudioJack_729JH
- added R30, R31: 47k, Resistor_SMD:R_0603_1608Metric, symbol Device:R
- added U12, U6, U9: DG442xY, Package_SO:SOIC-16_3.9x9.9mm_P1.27mm, symbol Analog_Switch:DG442xY
- R11: value 2k -> 4k7; LCSC C22975 -> C23162
- R17, R18: value 10k -> 47k; LCSC C25804 -> C25819
- R19, R20: value 300 -> 100; LCSC C17887 -> (none)
- R21: value 5k1 -> 47k; LCSC C23186 -> C25819
- R22: value 300 -> 47k; footprint Resistor_SMD:R_1206_3216Metric -> Resistor_SMD:R_0603_1608Metric; LCSC C17887 -> C25819
- RV1: footprint Potentiometer_THT:Potentiometer_Bourns_PDB_182_Dual_Horizontal_ReducedFootprint -> project_footprints:TRIM_PTN092-H10115K1B; symbol vca_backplane-rescue:R_POT_Dual-Device -> Device:R_Potentiometer_Dual; Bourns PDB182-K425K-103A -> (none); Digikey PDB182-K425K-103A -> PTN092-H10115K1A
- renumbered U14 to U10
Connections:
- net +12V: now also C14.1, U12.13 (V+), U6.13 (V+), U9.13 (V+); no longer C13.2
- net -12V: now also C13.2, U12.4 (V-), U6.4 (V-), U9.4 (V-); no longer C14.1
- net CARD1_OUT2: now also R17.2
- net CARD2_OUT2: now also R18.2
- net CARD3_OUT2: now also R21.2
- net CARD4_OUT2: now also R22.2
- net CARD5_OUT2: now also R30.2
- net CARD6_OUT2: now also R31.2
- net GND: now also U10.5 (+), J13.1, J9.1, U12.5 (GND), U6.5 (GND), U9.5 (GND); no longer U10.3 (+)
- net LEFT: now also J13.4
- net MIX1_CARD1_CTRL: now also U6.1
- net MIX1_CARD2_CTRL: now also U6.8
- net MIX1_CARD3_CTRL: now also U6.9
- net MIX1_CARD4_CTRL: now also U6.16
- net MIX1_CARD5_CTRL: now also U12.1
- net MIX1_CARD6_CTRL: now also U12.8
- net MIX1_VCA_IN: now also C27.1, R23.1, U12.3, U12.7, U6.11, U6.14, U6.3, U6.7
- net MIX2_VCA_IN: now also C28.1, R25.1, U12.11, U12.14, U9.11, U9.14, U9.3, U9.7
- net RIGHT: now also J9.4
- net at C20.1, R16.2, U7.13 (Io): now also U10.6 (-); no longer U10.2 (-)
- net at C19.2, R15.1, R19.2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: no longer R17.2
- net at C20.2, R16.1, R20.2: now also U10.7; no longer R18.2, U10.1
- net at R5.1: now also U6.2
- net at R7.1: now also U6.6
- net at R9.1: now also U6.10
- net at R12.1: now also U6.15
- net at R13.1: now also U12.2
- net at R14.1: now also U12.6
- net at R21.1: now also U9.2; no longer R22.2
- net MIX1_LEFT renamed MIX2_CARD2_CTRL
- net MIX2_CARD2_CTRL: now also U12.16
- net MIX1_RIGHT renamed MIX2_CARD1_CTRL
- net MIX2_CARD1_CTRL: now also U12.9
- net MIX2_A0 renamed MIX2_CARD4_CTRL
- net MIX2_CARD4_CTRL: now also U9.8
- net MIX2_A1 renamed MIX2_CARD5_CTRL
- net MIX2_CARD5_CTRL: now also U9.9
- net MIX2_A2 renamed MIX2_CARD6_CTRL
- net MIX2_CARD6_CTRL: now also U9.16
- net MIX2_SELECT_EN renamed MIX2_CARD3_CTRL
- net MIX2_CARD3_CTRL: now also U9.1
- net MONO: no longer names the net of R22.1
- net MONO: now also U9.6
- new net: R31.1, U9.15
- new net: R17.1, U12.10
- new net: R18.1, U12.15
- new net: R30.1, U9.10
- no-connect marks 14 -> 6
Other:
- note added: "DECOUPLING CAPS"
- note added: "OUTPUT VCA AND BUFFER"
- note removed: "DECOUPING CAPS"
- note removed: "LEFT/STEREO"
- note removed: "MIX1_LEFT MIX1_RIGHT : L R : NOTES 0 0 : MIX2 MIX2 : STEREO MIX2 0 1 : MIX2 MIX1 : DUAL MONO MIX2/MIX1 1 0 : MIX1 MIX2 : DUAL MONO MIX1/MIX2 1 1 : MIX1 MIX2 : STEREO MIX1"
- note removed: "Not Used"
- note removed: "Not quite as flexible as Mix1 by design: useful for stereo output of a single card or two independent outs"
- note removed: "OUTPUT SWITCHING"
- note removed: "RIGHT/MONO"
- moved on the sheet: C15, C16, C17, C18, C19, C20, C22, C23, C27, C28, C5, C7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

Commit message: starting on placement
Parts:
- R15, R16: footprint Resistor_SMD:R_0805_2012Metric -> Resistor_SMD:R_0603_1608Metric; LCSC C17713 -> C25819
- R23, R25: footprint Resistor_SMD:R_1206_3216Metric -> Resistor_SMD:R_0603_1608Metric; LCSC C17944 -> (none)
- U12, U6, U9: LCSC (none) -> C2673321
Connections:
- net LEFT: now also J13.3; no longer J13.4
- net RIGHT: now also J9.3; no longer J9.4
Changed lines of the file:
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@@
       (effects (font (size 1.27 1.27)))
     )
-    (property "Footprint" "Resistor_SMD:R_0805_2012Metric" (at 297.18 134.112 90)
+    (property "Footprint" "Resistor_SMD:R_0603_1608Metric" (at 297.18 134.112 90)
       (effects (font (size 1.27 1.27)) hide)
     )
@@
       (effects (font (size 1.27 1.27)) hide)
     )
-    (property "LCSC" "C17713" (at 297.18 135.89 0)
+    (property "LCSC" "C25819" (at 297.18 135.89 0)
       (effects (font (size 1.27 1.27)) hide)
     )
@@
       (effects (font (size 1.27 1.27)))
     )
-    (property "Footprint" "Resistor_SMD:R_0805_2012Metric" (at 298.45 173.482 90)
+    (property "Footprint" "Resistor_SMD:R_0603_1608Metric" (at 298.45 173.482 90)
       (effects (font (size 1.27 1.27)) hide)
     )
@@
       (effects (font (size 1.27 1.27)) hide)
     )
-    (property "LCSC" "C17713" (at 298.45 175.26 0)
+    (property "LCSC" "C25819" (at 298.45 175.26 0)
       (effects (font (size 1.27 1.27)) hide)
     )
@@
     )
     (property "Datasheet" "https://datasheets.maximintegrated.com/en/ds/DG441-DG442.pdf" (at 336.55 71.12 0)
+      (effects (font (size 1.27 1.27)) hide)
+    )
+    (property "LCSC" "C2673321" (at 336.55 71.12 0)
       (effects (font (size 1.27 1.27)) hide)
     )
@@
       (effects (font (size 1.27 1.27)) (justify left))
     )
-    (property "Footprint" "Resistor_SMD:R_1206_3216Metric" (at 257.302 160.02 90)
+    (property "Footprint" "Resistor_SMD:R_0603_1608Metric" (at 257.302 160.02 90)
       (effects (font (size 1.27 1.27)) hide)
     )
@@
       (effects (font (size 1.27 1.27)) hide)
     )
-    (property "LCSC" "C17944" (at 259.08 160.02 0)
+    (property "LCSC" "" (at 259.08 160.02 0)
       (effects (font (size 1.27 1.27)) hide)
     )
@@
     )
     (property "Datasheet" "https://datasheets.maximintegrated.com/en/ds/DG441-DG442.pdf" (at 336.55 31.75 0)
+      (effects (font (size 1.27 1.27)) hide)
+    )
+    (property "LCSC" "C2673321" (at 336.55 31.75 0)
       (effects (font (size 1.27 1.27)) hide)
     )
@@
       (effects (font (size 1.27 1.27)) hide)
     )
+    (property "LCSC" "C2673321" (at 196.85 33.02 0)
+      (effects (font (size 1.27 1.27)) hide)
+    )
     (pin "11")
     (pin "2")
@@
       (effects (font (size 1.27 1.27)) hide)
     )
+    (property "LCSC" "C2673321" (at 130.81 72.39 0)
+      (effects (font (size 1.27 1.27)) hide)
+    )
     (pin "11")
     (pin "2")
@@
       (effects (font (size 1.27 1.27)) hide)
     )
+    (property "LCSC" "C2673321" (at 130.81 53.34 0)
+      (effects (font (size 1.27 1.27)) hide)
+    )
     (pin "11")
     (pin "2")
@@
     )
     (property "Datasheet" "https://datasheets.maximintegrated.com/en/ds/DG441-DG442.pdf" (at 121.92 238.76 0)
+      (effects (font (size 1.27 1.27)) hide)
+    )
+    (property "LCSC" "C2673321" (at 121.92 238.76 0)
       (effects (font (size 1.27 1.27)) hide)
     )
@@
       (effects (font (size 1.27 1.27)) hide)
     )
+    (property "LCSC" "C2673321" (at 276.86 31.75 0)
+      (effects (font (size 1.27 1.27)) hide)
+    )
     (pin "15")
     (pin "5")
@@
       (effects (font (size 1.27 1.27)) hide)
     )
+    (property "LCSC" "C2673321" (at 196.85 53.34 0)
+      (effects (font (size 1.27 1.27)) hide)
+    )
     (pin "15")
     (pin "5")
@@
     )
     (property "Datasheet" "https://datasheets.maximintegrated.com/en/ds/DG441-DG442.pdf" (at 276.86 71.12 0)
+      (effects (font (size 1.27 1.27)) hide)
+    )
+    (property "LCSC" "C2673321" (at 276.86 71.12 0)
       (effects (font (size 1.27 1.27)) hide)
     )
@@
       (effects (font (size 1.27 1.27)) (justify left))
     )
-    (property "Footprint" "Resistor_SMD:R_1206_3216Metric" (at 254.762 198.12 90)
+    (property "Footprint" "Resistor_SMD:R_0603_1608Metric" (at 254.762 198.12 90)
       (effects (font (size 1.27 1.27)) hide)
     )
@@
       (effects (font (size 1.27 1.27)) hide)
     )
-    (property "LCSC" "C17944" (at 256.54 198.12 0)
+    (property "LCSC" "" (at 256.54 198.12 0)
       (effects (font (size 1.27 1.27)) hide)
     )
@@
     )
     (property "Datasheet" "https://datasheets.maximintegrated.com/en/ds/DG441-DG442.pdf" (at 196.85 72.39 0)
+      (effects (font (size 1.27 1.27)) hide)
+    )
+    (property "LCSC" "C2673321" (at 196.85 72.39 0)
       (effects (font (size 1.27 1.27)) hide)
     )
@@
       (effects (font (size 1.27 1.27)) hide)
     )
+    (property "LCSC" "C2673321" (at 66.04 238.76 0)
+      (effects (font (size 1.27 1.27)) hide)
+    )
     (pin "11")
     (pin "2")
@@
     )
     (property "Datasheet" "https://datasheets.maximintegrated.com/en/ds/DG441-DG442.pdf" (at 276.86 50.8 0)
+      (effects (font (size 1.27 1.27)) hide)
+    )
+    (property "LCSC" "C2673321" (at 276.86 50.8 0)
       (effects (font (size 1.27 1.27)) hide)
     )
@@
       (effects (font (size 1.27 1.27)) hide)
     )
+    (property "LCSC" "C2673321" (at 130.81 33.02 0)
+      (effects (font (size 1.27 1.27)) hide)
+    )
     (pin "11")
     (pin "2")
@@
     )
     (property "Datasheet" "https://datasheets.maximintegrated.com/en/ds/DG441-DG442.pdf" (at 336.55 50.8 0)
+      (effects (font (size 1.27 1.27)) hide)
+    )
+    (property "LCSC" "C2673321" (at 336.55 50.8 0)
       (effects (font (size 1.27 1.27)) hide)
     )
@@
       (effects (font (size 1.27 1.27)) hide)
     )
+    (property "LCSC" "C2673321" (at 93.98 238.76 0)
+      (effects (font (size 1.27 1.27)) hide)
+    )

Commit message: working on placement
Parts:
- removed TP15: TestPoint, TestPoint:TestPoint_Pad_2.0x2.0mm, symbol Connector:TestPoint
- renumbered R30 to R13, R13 to R30, U9 to U12, U9 to U6, U6 to U9, U12 to U9
Connections:
- net CARD1_OUT1: now also R17.2; no longer R5.2
- net CARD1_OUT2: now also R5.2; no longer R17.2
- net CARD3_OUT1: now also R21.2; no longer R9.2
- net CARD3_OUT2: now also R9.2; no longer R21.2
- net MIX1_CARD1_CTRL: now also U9.16; no longer U9.1
- net MIX1_CARD2_CTRL: now also U9.1; no longer U9.8
- net MIX1_CARD3_CTRL: now also U6.16; no longer U6.9
- net MIX1_CARD4_CTRL: now also U6.1; no longer U6.16
- net MIX1_CARD5_CTRL: now also U12.16; no longer U12.1
- net MIX1_CARD6_CTRL: now also U12.1; no longer U12.8
- net MIX1_VCA_IN: now also U12.14, U12.3, U6.14, U6.3, U9.14, U9.3; no longer U12.3, U12.7, U6.11, U6.14, U9.3, U9.7
- net MIX2_CARD2_CTRL: now also U9.8; no longer U9.16
- net MIX2_CARD3_CTRL: now also U6.9; no longer U6.1
- net MIX2_CARD6_CTRL: now also U12.8; no longer U12.16
- net MIX2_VCA_IN: now also U12.6, U6.11, U6.6, U9.6; no longer U12.14, U6.3, U6.7, U9.14
- net at R5.1: now also U9.10; no longer U9.2
- net at R7.1: now also U9.2; no longer U9.6
- net at R9.1: now also U6.10; no longer U6.10
- net at R12.1: now also U6.2; no longer U6.15
- net at R30.1: now also U12.15; no longer U12.2
- net at R14.1: now also U12.2; no longer U12.6
- net at R31.1: now also U12.7; no longer U12.15
- net at R17.1: now also U9.15; no longer U9.10
- net at R22.1: now also U6.7; no longer U6.6
- net at R18.1: now also U9.7; no longer U9.15
- net at R21.1: now also U6.15; no longer U6.2
Other:
- moved on the sheet: R17, R21, R5, R9, U12B, U6B, U9B
