File: kicad/vca_backplane/vca_backplane.kicad_sch (KiCad schematic)
At the start: 27 parts, among them J1 Conn_02x20_Odd_Even, J2 Eurorack Power, Q1 DMMT5401, Q2 DMG2305UX, U1 74HCT138, U11 74HCT138, U8 M24C02-WMN

Commit message: v0.2 of backplane submitted to jlcpcb
Parts:
- C1, C11, C12: LCSC (none) -> C14663; LCSC Part C14663 -> (none)
- Q1: LCSC (none) -> C154733; LCSC Part C154733 -> (none)
- Q2: LCSC (none) -> C150470; LCSC Part C150470 -> (none)
- R3: LCSC (none) -> C25804; LCSC Part C25804 -> (none)
- R6: LCSC (none) -> C25819; LCSC Part C25819 -> (none)
- U1, U11: LCSC (none) -> C8115; LCSC Part C8115 -> (none)
- U8: LCSC (none) -> C7562; LCSC Part C7562 -> (none)
Connections:
- net SPI_CLK_5V renamed SPI_CLK1_5V
- net SPI_MOSI_5V renamed SPI_MOSI1_5V
Other:
- sheet Level Shifting ports: added SPI_CLK1_5V, SPI_CLK2_5V, SPI_MOSI1_5V, SPI_MOSI2_5V; removed SPI_CLK_5V, SPI_MOSI_5V
- title: Raspberry Pi HAT -> Zoxnoxious Backplane and VCA
- moved on the sheet: TP3, TP4, TP5, TP6

Commit message: updates to 0.4 as3340 and 0.3 backplane
Parts:
- added J11: Conn_01x03, Connector_PinHeader_2.54mm:PinHeader_1x03_P2.54mm_Vertical, symbol Connector_Generic:Conn_01x03
- TP7: footprint TestPoint:TestPoint_Pad_2.0x2.0mm -> Connector_PinHeader_2.54mm:PinHeader_1x01_P2.54mm_Vertical
Connections:
- net GND: now also J11.1 (Pin_1)
- net RXD0: now reaches J1.10 (Pin_10)
- net RXD0: now also J11.3 (Pin_3)
- net TXD0: now reaches J1.8 (Pin_8)
- net TXD0: now also J11.2 (Pin_2)
- no-connect marks 20 -> 18
Other:
- note added: "Serial Console Interface"
- moved on the sheet: TP7
Changed lines of the file:
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@@
   (no_connect (at 154.94 196.85))
   (no_connect (at 138.43 259.08))
-  (no_connect (at 66.04 40.64))
-  (no_connect (at 66.04 38.1))
   (no_connect (at 222.25 199.39))
   (no_connect (at 210.82 196.85))
@@
     (stroke (width 0) (type default) (color 0 0 0 0))
   )
+  (wire (pts (xy 377.19 167.64) (xy 369.57 167.64))
+    (stroke (width 0) (type default) (color 0 0 0 0))
+  )
   (wire (pts (xy 303.53 182.88) (xy 320.04 182.88))
     (stroke (width 0) (type default) (color 0 0 0 0))
@@
     (stroke (width 0) (type default) (color 0 0 0 0))
   )
-  (wire (pts (xy 96.52 31.75) (xy 96.52 33.02))
+  (wire (pts (xy 379.73 151.13) (xy 379.73 152.4))
     (stroke (width 0) (type default) (color 0 0 0 0))
   )
@@
     (stroke (width 0) (type default) (color 0 0 0 0))
   )
+  (wire (pts (xy 66.04 38.1) (xy 85.09 38.1))
+    (stroke (width 0) (type default) (color 0 0 0 0))
+  )
   (wire (pts (xy 66.04 35.56) (xy 85.09 35.56))
     (stroke (width 0) (type default) (color 0 0 0 0))
@@
     (stroke (width 0) (type default) (color 0 0 0 0))
   )
+  (wire (pts (xy 377.19 165.1) (xy 369.57 165.1))
+    (stroke (width 0) (type default) (color 0 0 0 0))
+  )
   (wire (pts (xy 162.56 40.64) (xy 182.88 40.64))
     (stroke (width 0) (type default) (color 0 0 0 0))
@@
     (stroke (width 0) (type default) (color 0 0 0 0))
   )
+  (wire (pts (xy 377.19 170.18) (xy 369.57 170.18))
+    (stroke (width 0) (type default) (color 0 0 0 0))
+  )
   (wire (pts (xy 113.03 45.72) (xy 118.11 45.72))
     (stroke (width 0) (type default) (color 0 0 0 0))
@@
     (stroke (width 0) (type default) (color 0 0 0 0))
   )
+  (wire (pts (xy 66.04 40.64) (xy 85.09 40.64))
+    (stroke (width 0) (type default) (color 0 0 0 0))
+  )
   (wire (pts (xy 182.88 58.42) (xy 166.37 58.42))
     (stroke (width 0) (type default) (color 0 0 0 0))
@@
     (effects (font (size 1.524 1.524)) (justify left bottom))
   )
+  (text "Serial Console Interface" (at 372.11 173.99 0)
+    (effects (font (size 1.27 1.27)) (justify left bottom))
+  )
   (text "Chip Select w/ Level Shift" (at 114.3 160.02 0)
     (effects (font (size 2.54 2.54) (thickness 0.508) bold) (justify left bottom))
@@
     (effects (font (size 1.27 1.27)) (justify left bottom))
   )
+  (label "RXD0" (at 369.57 170.18 0)
+    (effects (font (size 1.27 1.27)) (justify left bottom))
+  )
   (label "GND" (at 85.09 45.72 180)
     (effects (font (size 1.524 1.524)) (justify right bottom))
@@
     (effects (font (size 1.27 1.27)) (justify left bottom))
   )
+  (label "RXD0" (at 85.09 40.64 180)
+    (effects (font (size 1.27 1.27)) (justify right bottom))
+  )
   (label "SCL_5V" (at 255.27 44.45 0)
     (effects (font (size 1.27 1.27)) (justify left bottom))
@@
     (effects (font (size 1.27 1.27)) (justify left bottom))
   )
+  (label "GND" (at 369.57 165.1 0)
+    (effects (font (size 1.27 1.27)) (justify left bottom))
+  )
   (label "MODULE_A_3V" (at 91.44 189.23 180)
     (effects (font (size 1.27 1.27)) (justify right bottom))
@@
     (effects (font (size 1.27 1.27)) (justify right bottom))
   )
+  (label "TXD0" (at 85.09 38.1 180)
+    (effects (font (size 1.27 1.27)) (justify right bottom))
+  )
   (label "SPI_CS1_D" (at 222.25 189.23 180)
     (effects (font (size 1.27 1.27)) (justify right bottom))
@@
     (effects (font (size 1.27 1.27)) (justify left bottom))
   )
+  (label "TXD0" (at 369.57 167.64 0)
+    (effects (font (size 1.27 1.27)) (justify left bottom))
+  )
   (label "SPI_CS1_C" (at 222.25 186.69 180)
     (effects (font (size 1.27 1.27)) (justify right bottom))
@@
     (pin "1")
   )
-  (symbol (lib_id "Connector:TestPoint") (at 96.52 31.75 0) (unit 1)
+  (symbol (lib_id "Connector:TestPoint") (at 379.73 151.13 0) (unit 1)
     (in_bom yes) (on_board yes)
-    (property "Reference" "TP7" (id 0) (at 97.9932 28.7528 0)
+    (property "Reference" "TP7" (id 0) (at 381.2032 148.1328 0)
       (effects (font (size 1.27 1.27)) (justify left))
     )
-    (property "Value" "TestPoint" (id 1) (at 97.9932 31.0642 0)
+    (property "Value" "TestPoint" (id 1) (at 381.2032 150.4442 0)
       (effects (font (size 1.27 1.27)) (justify left))
     )
-    (property "Footprint" "TestPoint:TestPoint_Pad_2.0x2.0mm" (id 2) (at 101.6 31.75 0)
+    (property "Footprint" "Connector_PinHeader_2.54mm:PinHeader_1x01_P2.54mm_Vertical" (id 2) (at 384.81 151.13 0)
       (effects (font (size 1.27 1.27)) hide)
     )
-    (property "Datasheet" "~" (id 3) (at 101.6 31.75 0)
+    (property "Datasheet" "~" (id 3) (at 384.81 151.13 0)
       (effects (font (size 1.27 1.27)) hide)
     )
-    (property "Digikey" "952-2664-2-ND" (id 4) (at 96.52 31.75 0)
+    (property "Digikey" "952-2664-2-ND" (id 4) (at 379.73 151.13 0)
       (effects (font (size 1.27 1.27)) hide)
     )
     (pin "1")
   )
-  (symbol (lib_id "power:GND") (at 96.52 33.02 0) (unit 1)
+  (symbol (lib_id "power:GND") (at 379.73 152.4 0) (unit 1)
     (in_bom yes) (on_board yes)
-    (property "Reference" "#PWR0171" (id 0) (at 96.52 39.37 0)
+    (property "Reference" "#PWR0171" (id 0) (at 379.73 158.75 0)
       (effects (font (size 1.27 1.27)) hide)
     )
-    (property "Value" "GND" (id 1) (at 96.52 36.83 0))
-    (property "Footprint" "" (id 2) (at 96.52 33.02 0))
-    (property "Datasheet" "" (id 3) (at 96.52 33.02 0))
+    (property "Value" "GND" (id 1) (at 379.73 156.21 0))
+    (property "Footprint" "" (id 2) (at 379.73 152.4 0))
+    (property "Datasheet" "" (id 3) (at 379.73 152.4 0))
     (pin "1")
   )
@@
     (pin "1")
   )
+  (symbol (lib_id "Connector_Generic:Conn_01x03") (at 382.27 167.64 0) (unit 1)
+    (in_bom yes) (on_board yes) (fields_autoplaced)
+    (property "Reference" "J11" (id 0) (at 384.302 166.8053 0)
+      (effects (font (size 1.27 1.27)) (justify left))
+    )
+    (property "Value" "Conn_01x03" (id 1) (at 384.302 169.3422 0)
+      (effects (font (size 1.27 1.27)) (justify left))
+    )
+    (property "Footprint" "Connector_PinHeader_2.54mm:PinHeader_1x03_P2.54mm_Vertical" (id 2) (at 382.27 167.64 0)
+      (effects (font (size 1.27 1.27)) hide)
+    )
+    (property "Datasheet" "~" (id 3) (at 382.27 167.64 0)
+      (effects (font (size 1.27 1.27)) hide)
+    )
+    (pin "1")
+    (pin "2")
+    (pin "3")
+  )
   (sheet (at 260.35 149.86) (size 43.18 57.15) (fields_autoplaced)
     (stroke (width 0) (type solid) (color 0 0 0 0))
@@
       (reference "J10") (unit 1) (value "AudioJack3DPDT") (footprint "Connector_Audio:Jack_6.35mm_CUI_SJ_63043F")
     )
+    (path "/7ed6a065-5e4e-4da2-b6f9-85f333a0c634"
+      (reference "J11") (unit 1) (value "Conn_01x03") (footprint "Connector_PinHeader_2.54mm:PinHeader_1x03_P2.54mm_Vertical")
+    )
     (path "/00000000-0000-0000-0000-000058e1538b"
       (reference "Q1") (unit 1) (value "DMMT5401") (footprint "Package_TO_SOT_SMD:SOT-23-6")
@@
     )
     (path "/00000000-0000-0000-0000-000063260b4c"
-      (reference "TP7") (unit 1) (value "TestPoint") (footprint "TestPoint:TestPoint_Pad_2.0x2.0mm")
+      (reference "TP7") (unit 1) (value "TestPoint") (footprint "Connector_PinHeader_2.54mm:PinHeader_1x01_P2.54mm_Vertical")
     )
     (path "/00000000-0000-0000-0000-00006309bcb4"

Commit message: schematic for backplane v0.3: change Pi GPIOs for SPI; switch output jacks; add external input
Parts:
- Q1: footprint Package_TO_SOT_SMD:SOT-23-6 -> SOT-26
Connections:
- net MUX_CS0: now also J1.38 (Pin_38); no longer J1.33 (Pin_33)
- net MUX_CS1: now also J1.40 (Pin_40); no longer J1.35 (Pin_35)
- net +3V3 renamed +3.3V
Other:
- added sheet external_input (external_input.kicad_sch)
- sheet sheet62525DC6 ports: added EXTERNAL; removed none
- sheet sheet6252A02B ports: added EXTERNAL; removed none
- sheet sheet6252A045 ports: added EXTERNAL; removed none
- sheet sheet625442EF ports: added EXTERNAL; removed none
- sheet sheet62544309 ports: added EXTERNAL; removed none
- sheet sheet62544323 ports: added EXTERNAL; removed none
- note added: "External Input"
- moved on the sheet: C11, J1, J11, J2, Q1A, Q1B, Q2, R3, R6, TP7, U8

Commit message: working on placement
Parts:
- Q1: footprint SOT-26 -> Package_TO_SOT_SMD:SOT-23-6
Connections:
- net MUX_CS1: now also J1.37 (Pin_37); no longer J1.40 (Pin_40)
- net MUX_CS2: now also J1.40 (Pin_40); no longer J1.37 (Pin_37)
Changed lines of the file:
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@@
   (junction (at 76.2 43.18) (diameter 0) (color 0 0 0 0)
   )
+  (junction (at 60.96 109.22) (diameter 0) (color 0 0 0 0)
+  )
   (junction (at 116.84 251.46) (diameter 0) (color 0 0 0 0)
   )
@@
   (junction (at 20.32 58.42) (diameter 0) (color 0 0 0 0)
   )
-  (junction (at 60.96 109.22) (diameter 0) (color 0 0 0 0)
-  )
   (junction (at 336.55 40.64) (diameter 0) (color 0 0 0 0)
   )
@@
     (stroke (width 0) (type default))
   )
-  (wire (pts (xy 60.96 109.22) (xy 77.47 109.22))
-    (stroke (width 0) (type default))
-  )
   (wire (pts (xy 270.51 83.82) (xy 254 83.82))
     (stroke (width 0) (type default))
@@
     (stroke (width 0) (type default))
   )
+  (wire (pts (xy 60.96 109.22) (xy 76.2 109.22))
+    (stroke (width 0) (type default))
+  )
   (wire (pts (xy 270.51 78.74) (xy 254 78.74))
     (stroke (width 0) (type default))
@@
     (effects (font (size 1.27 1.27)) (justify left bottom))
   )
-  (label "MUX_CS1" (at 71.12 76.2 180) (fields_autoplaced)
-    (effects (font (size 1.27 1.27)) (justify right bottom))
+  (label "MUX_CS1" (at 22.86 73.66 0) (fields_autoplaced)
+    (effects (font (size 1.27 1.27)) (justify left bottom))
   )
   (label "MUX_CS0" (at 71.12 73.66 180) (fields_autoplaced)
@@
     (effects (font (size 1.27 1.27)) (justify left bottom))
   )
-  (label "MUX_CS2" (at 22.86 73.66 0) (fields_autoplaced)
-    (effects (font (size 1.27 1.27)) (justify left bottom))
+  (label "MUX_CS2" (at 71.12 76.2 180) (fields_autoplaced)
+    (effects (font (size 1.27 1.27)) (justify right bottom))
   )
   (label "CARD6_OUT1" (at 414.02 114.3 180) (fields_autoplaced)
@@
       (effects (font (size 1.27 1.27)) (justify left))
     )
-    (property "Footprint" "SOT-26" (at 38.1 122.555 0)
+    (property "Footprint" "Package_TO_SOT_SMD:SOT-23-6" (at 38.1 122.555 0)
       (effects (font (size 1.27 1.27) italic) (justify left))
     )
@@
       (effects (font (size 1.27 1.27)) (justify left))
     )
-    (property "Footprint" "SOT-26" (at 63.5 122.555 0)
+    (property "Footprint" "Package_TO_SOT_SMD:SOT-23-6" (at 63.5 122.555 0)
       (effects (font (size 1.27 1.27) italic) (justify left))
     )
@@
         )
       )
-    )
-  )
-  (symbol (lib_id "power:PWR_FLAG") (at 77.47 109.22 0) (unit 1)
-    (in_bom yes) (on_board yes) (dnp no)
-    (property "Reference" "#FLG08" (at 77.47 107.315 0)
-      (effects (font (size 1.27 1.27)) hide)
-    )
-    (property "Value" "PWR_FLAG" (at 77.47 104.8258 0)
-      (effects (font (size 1.27 1.27)))
-    )
-    (property "Footprint" "" (at 77.47 109.22 0)
-      (effects (font (size 1.27 1.27)) hide)
-    )
-    (property "Datasheet" "~" (at 77.47 109.22 0)
-      (effects (font (size 1.27 1.27)) hide)
-    )
-    (pin "1")
-    (instances
-      (project "vca_backplane"
-        (path "/bdbd6910-8f28-459f-89ba-e6dd447d59a9"
-          (reference "#FLG08") (unit 1)
-        )
-      )

Commit message: tightening up placement
Parts:
- removed TP5: TestPoint, TestPoint:TestPoint_Pad_2.0x2.0mm, symbol Connector:TestPoint
- Q2: footprint Package_TO_SOT_SMD:SOT-23 -> project_footprints:SOT-23-DMG2305UX
Other:
- note removed: "Using SI2301CDS-T1-GE3 instead of spec’d DMG2305UX"
Changed lines of the file:
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@@
     (effects (font (size 2.9972 2.9972) (thickness 0.5994) bold) (justify left bottom))
-  )
-  (text "Using SI2301CDS-T1-GE3 instead of spec’d DMG2305UX"
-    (at 38.1 116.84 0)
-    (effects (font (size 1.27 1.27) (thickness 0.254) bold italic) (justify left bottom))
   )
   (text "Output Select" (at 384.81 157.48 0)
@@
       (effects (font (size 1.27 1.27)) (justify right))
     )
-    (property "Footprint" "Package_TO_SOT_SMD:SOT-23" (at 48.26 104.14 0)
-      (effects (font (size 1.27 1.27)) hide)
-    )
-    (property "Datasheet" "" (at 50.8 109.22 0)
-      (effects (font (size 1.27 1.27)))
+    (property "Footprint" "project_footprints:SOT-23-DMG2305UX" (at 48.26 104.14 0)
+      (effects (font (size 1.27 1.27)) hide)
+    )
+    (property "Datasheet" "https://jlcpcb.com/api/file/downloadByFileSystemAccessId/8560079443617075200" (at 50.8 109.22 0)
+      (effects (font (size 1.27 1.27)) hide)
     )
     (property "LCSC" "C150470" (at 50.8 109.22 0)
@@
         )
       )
-    )
-  )
-  (symbol (lib_id "Connector:TestPoint") (at 91.44 185.42 270) (unit 1)
-    (in_bom yes) (on_board yes) (dnp no)
-    (property "Reference" "TP5" (at 96.2152 184.2516 90)
-      (effects (font (size 1.27 1.27)) (justify left))
-    )
-    (property "Value" "TestPoint" (at 96.2152 186.563 90)
-      (effects (font (size 1.27 1.27)) (justify left))
-    )
-    (property "Footprint" "TestPoint:TestPoint_Pad_2.0x2.0mm" (at 91.44 190.5 0)
-      (effects (font (size 1.27 1.27)) hide)
-    )
-    (property "Datasheet" "~" (at 91.44 190.5 0)
-      (effects (font (size 1.27 1.27)) hide)
-    )
-    (property "Digikey" "952-2664-2-ND" (at 91.44 185.42 0)
-      (effects (font (size 1.27 1.27)) hide)
-    )
-    (pin "1")
-    (instances
-      (project "vca_backplane"
-        (path "/bdbd6910-8f28-459f-89ba-e6dd447d59a9"
-          (reference "TP5") (unit 1)
-        )
-      )
