File: kicad/poledancer/dac_2140.kicad_sch (KiCad schematic)
At the start: 16 parts, among them U7 AD5328

Commit message: geo reannotate
Parts:
- renumbered C14 to C23, C9 to C38, C13 to C39, C15 to C40, C16 to C41, C11 to C44, C12 to C45, R15 to R73, R11 to R74, R8 to R76, R9 to R77, R10 to R78, R14 to R79, R12 to R80, R13 to R81, U7 to U14
Changed lines of the file:
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@@
   (symbol (lib_id "Device:C") (at 224.79 85.09 0) (unit 1)
     (in_bom yes) (on_board yes) (dnp no)
-    (property "Reference" "C16" (at 220.345 84.455 0)
+    (property "Reference" "C41" (at 220.345 84.455 0)
       (effects (font (size 1.27 1.27)))
     )
@@
       (project "poledancer"
         (path "/7079bdb0-a00e-4bac-b257-cbcf2c91bbd6/a62c7733-d70d-462f-a319-1b36456deaa6"
-          (reference "C16") (unit 1)
+          (reference "C41") (unit 1)
         )
       )
@@
   (symbol (lib_id "Device:R") (at 201.93 58.42 270) (unit 1)
     (in_bom yes) (on_board yes) (dnp no)
-    (property "Reference" "R8" (at 200.025 53.975 90)
+    (property "Reference" "R76" (at 200.025 53.975 90)
       (effects (font (size 1.27 1.27)) (justify left))
     )
@@
       (project "poledancer"
         (path "/7079bdb0-a00e-4bac-b257-cbcf2c91bbd6/a62c7733-d70d-462f-a319-1b36456deaa6"
-          (reference "R8") (unit 1)
+          (reference "R76") (unit 1)
         )
       )
@@
   (symbol (lib_id "Device:R") (at 201.93 35.56 270) (unit 1)
     (in_bom yes) (on_board yes) (dnp no)
-    (property "Reference" "R9" (at 200.025 31.115 90)
+    (property "Reference" "R77" (at 200.025 31.115 90)
       (effects (font (size 1.27 1.27)) (justify left))
     )
@@
       (project "poledancer"
         (path "/7079bdb0-a00e-4bac-b257-cbcf2c91bbd6/a62c7733-d70d-462f-a319-1b36456deaa6"
-          (reference "R9") (unit 1)
+          (reference "R77") (unit 1)
         )
       )
@@
   (symbol (lib_id "Device:R") (at 201.93 80.01 270) (unit 1)
     (in_bom yes) (on_board yes) (dnp no)
-    (property "Reference" "R11" (at 200.025 75.565 90)
+    (property "Reference" "R74" (at 200.025 75.565 90)
       (effects (font (size 1.27 1.27)) (justify left))
     )
@@
       (project "poledancer"
         (path "/7079bdb0-a00e-4bac-b257-cbcf2c91bbd6/a62c7733-d70d-462f-a319-1b36456deaa6"
-          (reference "R11") (unit 1)
+          (reference "R74") (unit 1)
         )
       )
@@
   (symbol (lib_id "Device:R") (at 214.63 40.64 0) (unit 1)
     (in_bom yes) (on_board yes) (dnp no)
-    (property "Reference" "R13" (at 208.915 40.005 0)
+    (property "Reference" "R81" (at 208.915 40.005 0)
       (effects (font (size 1.27 1.27)) (justify left))
     )
@@
       (project "poledancer"
         (path "/7079bdb0-a00e-4bac-b257-cbcf2c91bbd6/a62c7733-d70d-462f-a319-1b36456deaa6"
-          (reference "R13") (unit 1)
+          (reference "R81") (unit 1)
         )
       )
@@
   (symbol (lib_id "Device:C") (at 46.99 64.77 0) (unit 1)
     (in_bom yes) (on_board yes) (dnp no)
-    (property "Reference" "C9" (at 42.545 64.135 0)
+    (property "Reference" "C38" (at 42.545 64.135 0)
       (effects (font (size 1.27 1.27)))
     )
@@
       (project "poledancer"
         (path "/7079bdb0-a00e-4bac-b257-cbcf2c91bbd6/a62c7733-d70d-462f-a319-1b36456deaa6"
-          (reference "C9") (unit 1)
+          (reference "C38") (unit 1)
         )
       )
@@
   (symbol (lib_id "Device:C") (at 224.79 40.64 0) (unit 1)
     (in_bom yes) (on_board yes) (dnp no)
-    (property "Reference" "C14" (at 220.345 40.005 0)
+    (property "Reference" "C23" (at 220.345 40.005 0)
       (effects (font (size 1.27 1.27)))
     )
@@
       (project "poledancer"
         (path "/7079bdb0-a00e-4bac-b257-cbcf2c91bbd6/a62c7733-d70d-462f-a319-1b36456deaa6"
-          (reference "C14") (unit 1)
+          (reference "C23") (unit 1)
         )
       )
@@
   (symbol (lib_id "Device:R") (at 214.63 63.5 0) (unit 1)
     (in_bom yes) (on_board yes) (dnp no)
-    (property "Reference" "R12" (at 208.915 62.865 0)
+    (property "Reference" "R80" (at 208.915 62.865 0)
       (effects (font (size 1.27 1.27)) (justify left))
     )
@@
       (project "poledancer"
         (path "/7079bdb0-a00e-4bac-b257-cbcf2c91bbd6/a62c7733-d70d-462f-a319-1b36456deaa6"
-          (reference "R12") (unit 1)
+          (reference "R80") (unit 1)
         )
       )
@@
   (symbol (lib_id "Device:C") (at 86.36 34.29 90) (unit 1)
     (in_bom yes) (on_board yes) (dnp no)
-    (property "Reference" "C11" (at 82.55 33.02 90)
+    (property "Reference" "C44" (at 82.55 33.02 90)
       (effects (font (size 1.27 1.27)))
     )
@@
       (project "poledancer"
         (path "/7079bdb0-a00e-4bac-b257-cbcf2c91bbd6/a62c7733-d70d-462f-a319-1b36456deaa6"
-          (reference "C11") (unit 1)
+          (reference "C44") (unit 1)
         )
       )
@@
   (symbol (lib_id "Device:C") (at 86.36 40.64 90) (unit 1)
     (in_bom yes) (on_board yes) (dnp no)
-    (property "Reference" "C12" (at 82.55 39.37 90)
+    (property "Reference" "C45" (at 82.55 39.37 90)
       (effects (font (size 1.27 1.27)))
     )
@@
       (project "poledancer"
         (path "/7079bdb0-a00e-4bac-b257-cbcf2c91bbd6/a62c7733-d70d-462f-a319-1b36456deaa6"
-          (reference "C12") (unit 1)
+          (reference "C45") (unit 1)
         )
       )
@@
   (symbol (lib_id "Device:C") (at 224.79 63.5 0) (unit 1)
     (in_bom yes) (on_board yes) (dnp no)
-    (property "Reference" "C13" (at 220.345 62.865 0)
+    (property "Reference" "C39" (at 220.345 62.865 0)
       (effects (font (size 1.27 1.27)))
     )
@@
       (project "poledancer"
         (path "/7079bdb0-a00e-4bac-b257-cbcf2c91bbd6/a62c7733-d70d-462f-a319-1b36456deaa6"
-          (reference "C13") (unit 1)
+          (reference "C39") (unit 1)
         )
       )
@@
   (symbol (lib_id "poledancer_symlib:AD5328") (at 77.47 58.42 0) (unit 1)
     (in_bom yes) (on_board yes) (dnp no)
-    (property "Reference" "U7" (at 76.2 58.42 0)
+    (property "Reference" "U14" (at 76.2 58.42 0)
       (effects (font (size 1.27 1.27)) (justify left))
     )
@@
       (project "poledancer"
         (path "/7079bdb0-a00e-4bac-b257-cbcf2c91bbd6/a62c7733-d70d-462f-a319-1b36456deaa6"
-          (reference "U7") (unit 1)
+          (reference "U14") (unit 1)
         )
       )
@@
   (symbol (lib_id "Device:R") (at 214.63 107.95 0) (unit 1)
     (in_bom yes) (on_board yes) (dnp no)
-    (property "Reference" "R14" (at 208.915 107.315 0)
+    (property "Reference" "R79" (at 208.915 107.315 0)
       (effects (font (size 1.27 1.27)) (justify left))
     )
@@
       (project "poledancer"
         (path "/7079bdb0-a00e-4bac-b257-cbcf2c91bbd6/a62c7733-d70d-462f-a319-1b36456deaa6"
-          (reference "R14") (unit 1)
+          (reference "R79") (unit 1)
         )
       )
@@
   (symbol (lib_id "Device:C") (at 224.79 107.95 0) (unit 1)
     (in_bom yes) (on_board yes) (dnp no)
-    (property "Reference" "C15" (at 220.345 107.315 0)
+    (property "Reference" "C40" (at 220.345 107.315 0)
       (effects (font (size 1.27 1.27)))
     )
@@
       (project "poledancer"
         (path "/7079bdb0-a00e-4bac-b257-cbcf2c91bbd6/a62c7733-d70d-462f-a319-1b36456deaa6"
-          (reference "C15") (unit 1)
+          (reference "C40") (unit 1)
         )
       )
@@
   (symbol (lib_id "Device:R") (at 214.63 85.09 0) (unit 1)
     (in_bom yes) (on_board yes) (dnp no)
-    (property "Reference" "R15" (at 208.915 84.455 0)
+    (property "Reference" "R73" (at 208.915 84.455 0)
       (effects (font (size 1.27 1.27)) (justify left))
     )
@@
       (project "poledancer"
         (path "/7079bdb0-a00e-4bac-b257-cbcf2c91bbd6/a62c7733-d70d-462f-a319-1b36456deaa6"
-          (reference "R15") (unit 1)
+          (reference "R73") (unit 1)
         )
       )
@@
   (symbol (lib_id "Device:R") (at 201.93 102.87 270) (unit 1)
     (in_bom yes) (on_board yes) (dnp no)
-    (property "Reference" "R10" (at 200.025 98.425 90)
+    (property "Reference" "R78" (at 200.025 98.425 90)
       (effects (font (size 1.27 1.27)) (justify left))
     )
@@
       (project "poledancer"
         (path "/7079bdb0-a00e-4bac-b257-cbcf2c91bbd6/a62c7733-d70d-462f-a319-1b36456deaa6"
-          (reference "R10") (unit 1)
-        )
-      )
+          (reference "R78") (unit 1)
+        )
+      )
